Commit message: #23 First version of somehow working hardware interface

File: elkapod_description/ros2_control/legs_system.ros2_control.xacro (robot description, xacro)
@@ -7,6 +7,5 @@
     </joint>
   </xacro:macro>
-  <xacro:macro name="legs_system_ros2_control" params="name prefix use_mock_hardware">
-    <ros2_control name="${name}" type="system">
+  <ros2_control name="ElkapodLegsSystemHardware" type="system">
       <hardware>
           <plugin>elkapod_description/ElkapodLegsSystemHardware</plugin>
@@ -33,5 +32,4 @@
       <xacro:joint_interface name="leg6_J2"/>
       <xacro:joint_interface name="leg6_J3"/>
-    </ros2_control>
-  </xacro:macro>
+  </ros2_control>
 </robot>

File: elkapod_description/urdf/elkapod.urdf.xacro (robot description, xacro)
@@ -21,4 +21,4 @@
   <xacro:include filename="$(find elkapod_description)/urdf/imu.xacro" />
   <!-- ros2_control -->
-  <xacro:include filename="$(find elkapod_description)/ros2_control/sim_system.ros2_control.xacro" />
+  <xacro:include filename="$(find elkapod_description)/ros2_control/legs_system.ros2_control.xacro" />
 </robot>
