Commit message: Added using sim_time for all walking stack nodes, unification of hardware and simulation joint interfaces, typo fixes

File: elkapod_description/ros2_control/elkapod.ros2_control.xacro (robot description, xacro)
@@ -2,13 +2,8 @@
 <robot xmlns:xacro="http://www.ros.org/wiki/xacro">
     <!-- Sim mode joint definition -->
-    <xacro:macro name="sim_joint_interface" params="name min_pos_rad max_pos_rad initial_angle_rad">
+    <xacro:macro name="sim_joint_interface" params="name">
         <joint name="${name}">
-            <command_interface name="position">
-            <param name="min">${min_pos_rad}</param>
-            <param name="max">${max_pos_rad}</param>
-            </command_interface>
-            <state_interface name="position">
-                <param name="initial_value">${initial_angle_rad}</param>
-            </state_interface>
+            <command_interface name="position"/>
+            <state_interface name="position"/>
             <state_interface name="velocity"/>
             <state_interface name="effort"/>
@@ -47,22 +42,22 @@
                     <plugin>gz_ros2_control/GazeboSimSystem</plugin>
                 </hardware>
-                <xacro:sim_joint_interface name="leg1_J1" min_pos_rad="-1.57" max_pos_rad="1.57" initial_angle_rad="0.0"/>
-                <xacro:sim_joint_interface name="leg1_J2" min_pos_rad="-1.57" max_pos_rad="1.57" initial_angle_rad="0.0"/>
-                <xacro:sim_joint_interface name="leg1_J3" min_pos_rad="-3.14" max_pos_rad="0.0" initial_angle_rad="0.0"/>
-                <xacro:sim_joint_interface name="leg3_J1" min_pos_rad="-1.57" max_pos_rad="1.57" initial_angle_rad="0.0"/>
-                <xacro:sim_joint_interface name="leg3_J2" min_pos_rad="-1.57" max_pos_rad="1.57" initial_angle_rad="0.0"/>
-                <xacro:sim_joint_interface name="leg3_J3" min_pos_rad="-3.14" max_pos_rad="0.0" initial_angle_rad="0.0"/>
-                <xacro:sim_joint_interface name="leg5_J1" min_pos_rad="-1.57" max_pos_rad="1.57" initial_angle_rad="0.0"/>
-                <xacro:sim_joint_interface name="leg5_J2" min_pos_rad="-1.57" max_pos_rad="1.57" initial_angle_rad="0.0"/>
-                <xacro:sim_joint_interface name="leg5_J3" min_pos_rad="-3.14" max_pos_rad="0.0" initial_angle_rad="0.0"/>
-                <xacro:sim_joint_interface name="leg2_J1" min_pos_rad="-1.57" max_pos_rad="1.57" initial_angle_rad="0.0"/>
-                <xacro:sim_joint_interface name="leg2_J2" min_pos_rad="-1.57" max_pos_rad="1.57" initial_angle_rad="0.0"/>
-                <xacro:sim_joint_interface name="leg2_J3" min_pos_rad="-3.14" max_pos_rad="0.0" initial_angle_rad="0.0"/>
-                <xacro:sim_joint_interface name="leg4_J1" min_pos_rad="-1.57" max_pos_rad="1.57" initial_angle_rad="0.0"/>
-                <xacro:sim_joint_interface name="leg4_J2" min_pos_rad="-1.57" max_pos_rad="1.57" initial_angle_rad="0.0"/>
-                <xacro:sim_joint_interface name="leg4_J3" min_pos_rad="-3.14" max_pos_rad="0.0" initial_angle_rad="0.0"/>
-                <xacro:sim_joint_interface name="leg6_J1" min_pos_rad="-1.57" max_pos_rad="1.57" initial_angle_rad="0.0"/>
-                <xacro:sim_joint_interface name="leg6_J2" min_pos_rad="-1.57" max_pos_rad="1.57" initial_angle_rad="0.0"/>
-                <xacro:sim_joint_interface name="leg6_J3" min_pos_rad="-3.14" max_pos_rad="0.0" initial_angle_rad="0.0"/>
+                <xacro:sim_joint_interface name="leg1_J1"/>
+                <xacro:sim_joint_interface name="leg1_J2"/>
+                <xacro:sim_joint_interface name="leg1_J3"/>
+                <xacro:sim_joint_interface name="leg3_J1"/>
+                <xacro:sim_joint_interface name="leg3_J2"/>
+                <xacro:sim_joint_interface name="leg3_J3"/>
+                <xacro:sim_joint_interface name="leg5_J1"/>
+                <xacro:sim_joint_interface name="leg5_J2"/>
+                <xacro:sim_joint_interface name="leg5_J3"/>
+                <xacro:sim_joint_interface name="leg2_J1"/>
+                <xacro:sim_joint_interface name="leg2_J2"/>
+                <xacro:sim_joint_interface name="leg2_J3"/>
+                <xacro:sim_joint_interface name="leg4_J1"/>
+                <xacro:sim_joint_interface name="leg4_J2"/>
+                <xacro:sim_joint_interface name="leg4_J3"/>
+                <xacro:sim_joint_interface name="leg6_J1"/>
+                <xacro:sim_joint_interface name="leg6_J2"/>
+                <xacro:sim_joint_interface name="leg6_J3"/>
             </ros2_control>
             <!-- IMU simulation setup -->

Commit message: Closes #32, added new parameters for better leg traction to the surface

File: elkapod_description/ros2_control/elkapod.ros2_control.xacro (robot description, xacro)
@@ -5,4 +5,11 @@
         <joint name="${name}">
             <command_interface name="position"/>
+            <state_interface name="position"/>
+            <state_interface name="velocity"/>
+            <state_interface name="effort"/>
+        </joint>
+    </xacro:macro>
+    <xacro:macro name="sim_fcp_joint_interface" params="name">
+        <joint name="${name}">
             <state_interface name="position"/>
             <state_interface name="velocity"/>
@@ -60,4 +67,11 @@
                 <xacro:sim_joint_interface name="leg6_J2"/>
                 <xacro:sim_joint_interface name="leg6_J3"/>
+                <!-- FCP joints (only for joint states broadcaster)-->
+                <xacro:sim_fcp_joint_interface name="leg1_FCP_joint"/>
+                <xacro:sim_fcp_joint_interface name="leg2_FCP_joint"/>
+                <xacro:sim_fcp_joint_interface name="leg3_FCP_joint"/>
+                <xacro:sim_fcp_joint_interface name="leg4_FCP_joint"/>
+                <xacro:sim_fcp_joint_interface name="leg5_FCP_joint"/>
+                <xacro:sim_fcp_joint_interface name="leg6_FCP_joint"/>
             </ros2_control>
             <!-- IMU simulation setup -->

File: elkapod_description/urdf/left_leg/left_leg.urdf.xacro (robot description, xacro)
@@ -140,6 +140,9 @@
     </link>
     <gazebo reference="${leg_name}_FCP">
-      <mu1>10.0</mu1>
-      <mu2>10.0</mu2>
+      <mu1>0.8</mu1>
+      <mu2>0.8</mu2>
+      <kp>1000000.0</kp>
+      <kd>100.0</kd>
+      <minDepth>0.01</minDepth>
     </gazebo>
     <gazebo reference="${leg_name}_FCP_joint">
@@ -148,5 +151,5 @@
           <update_rate>100</update_rate>
           <visualize>true</visualize>
-          <topic>/legs/${leg_name}/fsr</topic>
+          <topic>/legs/${leg_name}_fsr</topic>
           <enable_metrics>true</enable_metrics>
           <pose>0 0 0 0 0 0</pose>

File: elkapod_description/urdf/right_leg/right_leg.urdf.xacro (robot description, xacro)
@@ -140,6 +140,9 @@
     </link>
     <gazebo reference="${leg_name}_FCP">
-      <mu1>10.0</mu1>
-      <mu2>10.0</mu2>
+      <mu1>0.8</mu1>
+      <mu2>0.8</mu2>
+      <kp>1000000.0</kp>
+      <kd>100.0</kd>
+      <minDepth>0.01</minDepth>
     </gazebo>
     <gazebo reference="${leg_name}_FCP_joint">
@@ -148,5 +151,5 @@
           <update_rate>100</update_rate>
           <visualize>true</visualize>
-          <topic>/legs/${leg_name}/fsr</topic>
+          <topic>/legs/${leg_name}_fsr</topic>
           <enable_metrics>true</enable_metrics>
           <pose>0 0 0 0 0 0</pose>

Commit message: Walking stack v1.5.0 (#40)
* Increased trajectory frequency for motion manager, fixed bug in motion manager config

* Added using sim_time for all walking stack nodes, unification of hardware and simulation joint interfaces, typo fixes

* #37 Added parameter to controller manager launch enforcing joint limits

* #19 Started implementing inverse kinematics controller

* #33 #35 Started implementing new gait, smoother gait generator algorithm, rotation not working for now

* #33 #35 Temporarly fixed setting angular velocity for the robot

* #33 #35 Finalized input velocity commands pipeline, cleaned code

* #39 Implemented RIPPLE gait, changed order of leg movement during stand up phase in motion manager

* Fixed Werror errors during compilation

* #32 First version of force sensors added

* Closes #32, added new parameters for better leg traction to the surface

* #19 #33 Added pose correction, IK controller arguments passing, changed feet friction

* Changed launch for hardware

* Removed passthrough controller

* Fixed parameters passing, updated stand up sequence

* Fixed #24

* Refactored code for LegPath, cleaned Gait generator code

* Removed elkapod_gait_gen_py

* Updated elkapod_gait_gen_cpp version

* Test stand up sequence for 4 legs

File: elkapod_description/ros2_control/elkapod.ros2_control.xacro (robot description, xacro)
@@ -2,13 +2,15 @@
 <robot xmlns:xacro="http://www.ros.org/wiki/xacro">
     <!-- Sim mode joint definition -->
-    <xacro:macro name="sim_joint_interface" params="name min_pos_rad max_pos_rad initial_angle_rad">
+    <xacro:macro name="sim_joint_interface" params="name">
         <joint name="${name}">
-            <command_interface name="position">
-            <param name="min">${min_pos_rad}</param>
-            <param name="max">${max_pos_rad}</param>
-            </command_interface>
-            <state_interface name="position">
-                <param name="initial_value">${initial_angle_rad}</param>
-            </state_interface>
+            <command_interface name="position"/>
+            <state_interface name="position"/>
+            <state_interface name="velocity"/>
+            <state_interface name="effort"/>
+        </joint>
+    </xacro:macro>
+    <xacro:macro name="sim_fcp_joint_interface" params="name">
+        <joint name="${name}">
+            <state_interface name="position"/>
             <state_interface name="velocity"/>
             <state_interface name="effort"/>
@@ -34,5 +36,5 @@
                 <plugin name="gz_ros2_control::GazeboSimROS2ControlPlugin" filename="libgz_ros2_control-system.so">
                     <parameters>$(find elkapod_description)/config/my_controllers.yaml</parameters>
-                    <parameters>$(find elkapod_description)/config/gaz_ros2_ctl_use_sim.yaml</parameters>
+                    <!-- <parameters>$(find elkapod_description)/config/gaz_ros2_ctl_use_sim.yaml</parameters> -->
                 </plugin>
                 <plugin filename="gz-sim-odometry-publisher-system" name="gz::sim::systems::OdometryPublisher">
@@ -47,22 +49,29 @@
                     <plugin>gz_ros2_control/GazeboSimSystem</plugin>
                 </hardware>
-                <xacro:sim_joint_interface name="leg1_J1" min_pos_rad="-1.57" max_pos_rad="1.57" initial_angle_rad="0.0"/>
-                <xacro:sim_joint_interface name="leg1_J2" min_pos_rad="-1.57" max_pos_rad="1.57" initial_angle_rad="0.0"/>
-                <xacro:sim_joint_interface name="leg1_J3" min_pos_rad="-3.14" max_pos_rad="0.0" initial_angle_rad="0.0"/>
-                <xacro:sim_joint_interface name="leg3_J1" min_pos_rad="-1.57" max_pos_rad="1.57" initial_angle_rad="0.0"/>
-                <xacro:sim_joint_interface name="leg3_J2" min_pos_rad="-1.57" max_pos_rad="1.57" initial_angle_rad="0.0"/>
-                <xacro:sim_joint_interface name="leg3_J3" min_pos_rad="-3.14" max_pos_rad="0.0" initial_angle_rad="0.0"/>
-                <xacro:sim_joint_interface name="leg5_J1" min_pos_rad="-1.57" max_pos_rad="1.57" initial_angle_rad="0.0"/>
-                <xacro:sim_joint_interface name="leg5_J2" min_pos_rad="-1.57" max_pos_rad="1.57" initial_angle_rad="0.0"/>
-                <xacro:sim_joint_interface name="leg5_J3" min_pos_rad="-3.14" max_pos_rad="0.0" initial_angle_rad="0.0"/>
-                <xacro:sim_joint_interface name="leg2_J1" min_pos_rad="-1.57" max_pos_rad="1.57" initial_angle_rad="0.0"/>
-                <xacro:sim_joint_interface name="leg2_J2" min_pos_rad="-1.57" max_pos_rad="1.57" initial_angle_rad="0.0"/>
-                <xacro:sim_joint_interface name="leg2_J3" min_pos_rad="-3.14" max_pos_rad="0.0" initial_angle_rad="0.0"/>
-                <xacro:sim_joint_interface name="leg4_J1" min_pos_rad="-1.57" max_pos_rad="1.57" initial_angle_rad="0.0"/>
-                <xacro:sim_joint_interface name="leg4_J2" min_pos_rad="-1.57" max_pos_rad="1.57" initial_angle_rad="0.0"/>
-                <xacro:sim_joint_interface name="leg4_J3" min_pos_rad="-3.14" max_pos_rad="0.0" initial_angle_rad="0.0"/>
-                <xacro:sim_joint_interface name="leg6_J1" min_pos_rad="-1.57" max_pos_rad="1.57" initial_angle_rad="0.0"/>
-                <xacro:sim_joint_interface name="leg6_J2" min_pos_rad="-1.57" max_pos_rad="1.57" initial_angle_rad="0.0"/>
-                <xacro:sim_joint_interface name="leg6_J3" min_pos_rad="-3.14" max_pos_rad="0.0" initial_angle_rad="0.0"/>
+                <xacro:sim_joint_interface name="leg1_J1"/>
+                <xacro:sim_joint_interface name="leg1_J2"/>
+                <xacro:sim_joint_interface name="leg1_J3"/>
+                <xacro:sim_joint_interface name="leg3_J1"/>
+                <xacro:sim_joint_interface name="leg3_J2"/>
+                <xacro:sim_joint_interface name="leg3_J3"/>
+                <xacro:sim_joint_interface name="leg5_J1"/>
+                <xacro:sim_joint_interface name="leg5_J2"/>
+                <xacro:sim_joint_interface name="leg5_J3"/>
+                <xacro:sim_joint_interface name="leg2_J1"/>
+                <xacro:sim_joint_interface name="leg2_J2"/>
+                <xacro:sim_joint_interface name="leg2_J3"/>
+                <xacro:sim_joint_interface name="leg4_J1"/>
+                <xacro:sim_joint_interface name="leg4_J2"/>
+                <xacro:sim_joint_interface name="leg4_J3"/>
+                <xacro:sim_joint_interface name="leg6_J1"/>
+                <xacro:sim_joint_interface name="leg6_J2"/>
+                <xacro:sim_joint_interface name="leg6_J3"/>
+                <!-- FCP joints (only for joint states broadcaster)-->
+                <xacro:sim_fcp_joint_interface name="leg1_FCP_joint"/>
+                <xacro:sim_fcp_joint_interface name="leg2_FCP_joint"/>
+                <xacro:sim_fcp_joint_interface name="leg3_FCP_joint"/>
+                <xacro:sim_fcp_joint_interface name="leg4_FCP_joint"/>
+                <xacro:sim_fcp_joint_interface name="leg5_FCP_joint"/>
+                <xacro:sim_fcp_joint_interface name="leg6_FCP_joint"/>
             </ros2_control>
             <!-- IMU simulation setup -->

File: elkapod_description/urdf/left_leg/left_leg.urdf.xacro (robot description, xacro)
@@ -142,11 +142,30 @@
       <mu1>10.0</mu1>
       <mu2>10.0</mu2>
+      <kp>1000000.0</kp>
+      <kd>100.0</kd>
+      <minDepth>0.01</minDepth>
+    </gazebo>
+    <gazebo reference="${leg_name}_FCP_joint">
+        <sensor name="${leg_name}_fsr" type="force_torque">
+          <always_on>true</always_on>
+          <update_rate>100</update_rate>
+          <visualize>true</visualize>
+          <topic>/legs/${leg_name}_fsr</topic>
+          <enable_metrics>true</enable_metrics>
+          <pose>0 0 0 0 0 0</pose>
+          <force_torque>
+            <frame>sensor</frame>
+            <measure_direction>child_to_parent</measure_direction>
+          </force_torque>
+        </sensor>
     </gazebo>
     <!-- Fixed Joint for FCP -->
-    <joint name="${leg_name}_FCP_joint" type="fixed">
+    <joint name="${leg_name}_FCP_joint" type="prismatic">
       <origin xyz="0.2135 0.0085747 0" rpy="0 0 -0.29403" />
       <parent link="${leg_name}_linkC" />
       <child link="${leg_name}_FCP" />
-      <axis xyz="0 0 0" />
+      <axis xyz="1 0 0" />
+      <limit effort="1000.0" lower="-0.0001" upper="0.0001" velocity="30"/>
+      <dynamics damping="10.0" friction="0.0"/>
     </joint>
   </xacro:macro>

File: elkapod_description/urdf/right_leg/right_leg.urdf.xacro (robot description, xacro)
@@ -142,11 +142,30 @@
       <mu1>10.0</mu1>
       <mu2>10.0</mu2>
+      <kp>1000000.0</kp>
+      <kd>100.0</kd>
+      <minDepth>0.01</minDepth>
+    </gazebo>
+    <gazebo reference="${leg_name}_FCP_joint">
+        <sensor name="${leg_name}_fsr" type="force_torque">
+          <always_on>true</always_on>
+          <update_rate>100</update_rate>
+          <visualize>true</visualize>
+          <topic>/legs/${leg_name}_fsr</topic>
+          <enable_metrics>true</enable_metrics>
+          <pose>0 0 0 0 0 0</pose>
+          <force_torque>
+            <frame>sensor</frame>
+            <measure_direction>child_to_parent</measure_direction>
+          </force_torque>
+        </sensor>
     </gazebo>
     <!-- Fixed joint for FCP -->
-    <joint name="${leg_name}_FCP_joint" type="fixed">
+    <joint name="${leg_name}_FCP_joint" type="prismatic">
         <origin xyz="0.213503787197785 0.00857470533092818 0" rpy="0 0 -0.294032099334707" />
         <parent link="${leg_name}_linkC" />
         <child link="${leg_name}_FCP" />
-        <axis xyz="0 0 0" />
+        <axis xyz="1 0 0" />
+        <limit effort="1000.0" lower="-0.0001" upper="0.0001" velocity="30"/>
+        <dynamics damping="10.0" friction="0.0"/>
     </joint>
   </xacro:macro>
