Commit message: Finished tuning sensor parameters

File: elkapod_description/urdf/sensors/depth_camera.xacro (robot description, xacro)
@@ -28,8 +28,7 @@
         <axis xyz="0 0 0" />
     </joint>
-    <!-- Probably unnecessary, but will keep it for now-->
     <link name="front_camera_optical"></link>
     <joint name="front_camera_optical_fixed" type="fixed">
-        <origin xyz="0 0 0" rpy="0 0 0" />
+        <origin xyz="0 0 0" rpy="3.14159265359  0 0" />
         <parent link="front_camera_link" />
         <child link="front_camera_optical" />
@@ -41,18 +40,26 @@
             <topic>front_camera</topic>
             <visualize>true</visualize>
-            <update_rate>10</update_rate>
+            <update_rate>30</update_rate>
             <always_on>true</always_on>
             <camera>
-                <camera_horizontal_fov>1</camera_horizontal_fov>
+                <horizontal_fov>1.20428</horizontal_fov>
                 <image>
                     <format>R8G8B8</format>
-                    <width>320</width>
-                    <height>240</height>
+                    <width>640</width>
+                    <height>480</height>
                 </image>
                 <clip>
-                    <near>0.2</near>
+                    <near>0.1</near>
                     <far>30</far>
                 </clip>
+                <depth_camera>
+                    <output>depths</output>
+                    <clip>
+                        <near>0.1</near>
+                        <far>30</far>
+                    </clip>
+                </depth_camera>
             </camera>
+            <gz_frame_id>front_camera_optical</gz_frame_id>
         </sensor>
     </gazebo>

File: elkapod_description/urdf/sensors/lidar.xacro (robot description, xacro)
@@ -38,5 +38,7 @@
         <sensor name="lidar" type="gpu_lidar">
             <always_on>true</always_on>
-            <update_rate>2</update_rate>
+            <!-- Downgraded values, so your GPU doesn't melt -->
+            <!-- <update_rate>10</update_rate> -->
+            <update_rate>3</update_rate>
             <visualize>true</visualize>
             <topic>lidar_data</topic>
@@ -44,5 +46,7 @@
                 <scan>
                     <horizontal>
-                        <samples>45</samples>
+                        <!-- Downgraded values, so your GPU doesn't melt -->
+                        <!-- <samples>900</samples> -->
+                        <samples>90</samples>
                         <resolution>1</resolution>
                         <min_angle>-3.14</min_angle>
@@ -50,14 +54,16 @@
                     </horizontal>
                     <vertical>
+                        <!-- Downgraded values, so your GPU doesn't melt -->
                         <samples>25</samples>
+                        <!-- <samples>95</samples> -->
                         <resolution>1</resolution>
                         <min_angle>0</min_angle>
-                        <max_angle>1.3</max_angle>
+                        <max_angle>1.57079633</max_angle>
                     </vertical>
                 </scan>
                 <range>
-                    <min>0.05</min>
-                    <max>20</max>
-                    <resolution>0.005</resolution>
+                    <min>0.1</min>
+                    <max>30</max>
+                    <resolution>0.01</resolution>
                 </range>
             </lidar>
