Commit message: Added ros2 control, imu sensor

File: elkapod_description/urdf/body/body.urdf.xacro (robot description, xacro)
@@ -1,6 +1,14 @@
 <?xml version="1.0" encoding="utf-8"?>
 <robot xmlns:xacro="http://ros.org/wiki/xacro">
+  <!-- BASE LINK -->
+    <link name="base_link">
+  </link>
+  <joint name="base_body_link" type="fixed">
+        <parent link="base_link"/>
+        <child link="body_link"/>
+        <origin xyz="0 0 0" rpy="0 0 0"/>
+  </joint>
   <link
-    name="base_link">
+    name="body_link">
     <inertial>
       <origin

File: elkapod_description/urdf/elkapod.urdf.xacro (robot description, xacro)
@@ -11,9 +11,12 @@
   <xacro:include filename="$(find elkapod_description)/urdf/left_leg/left_leg.urdf.xacro" />
   <xacro:include filename="$(find elkapod_description)/urdf/right_leg/right_leg.urdf.xacro" />
-  <xacro:leg_left leg_name="leg1" parent="base_link" pos_x="0.13" pos_y="0.13" pos_z="-0.025" roll="0" pitch="0" yaw="1.57"/>
-  <xacro:leg_left leg_name="leg3" parent="base_link" pos_x="0.0" pos_y="0.13" pos_z="-0.025" roll="0" pitch="0" yaw="1.57"/>
-  <xacro:leg_left leg_name="leg5" parent="base_link" pos_x="-0.13" pos_y="0.13" pos_z="-0.025" roll="0" pitch="0" yaw="1.57"/>
-  <xacro:leg_right leg_name="leg2" parent="base_link" pos_x="0.13" pos_y="-0.13" pos_z="-0.025" roll="0" pitch="0" yaw="-1.57"/>
-  <xacro:leg_right leg_name="leg4" parent="base_link" pos_x="0.0" pos_y="-0.13" pos_z="-0.025" roll="0" pitch="0" yaw="-1.57"/>
-  <xacro:leg_right leg_name="leg6" parent="base_link" pos_x="-0.13" pos_y="-0.13" pos_z="-0.025" roll="0" pitch="0" yaw="-1.57"/>
+  <xacro:leg_left leg_name="leg1" parent="base_link" pos_x="0.17841" pos_y="0.13276" pos_z="-0.03" roll="0" pitch="0" yaw="0.63973287"/>
+  <xacro:leg_left leg_name="leg3" parent="base_link" pos_x="0.0138" pos_y="0.1643" pos_z="-0.03" roll="0" pitch="0" yaw="1.57"/>
+  <xacro:leg_left leg_name="leg5" parent="base_link" pos_x="-0.15903" pos_y="0.15038" pos_z="-0.03" roll="0" pitch="0" yaw="2.384143643587"/>
+  <xacro:leg_right leg_name="leg2" parent="base_link" pos_x="0.17841" pos_y="-0.13276" pos_z="-0.03" roll="0" pitch="0" yaw="-0.63973287"/>
+  <xacro:leg_right leg_name="leg4" parent="base_link" pos_x="0.0138" pos_y="-0.1643" pos_z="-0.03" roll="0" pitch="0" yaw="-1.57"/>
+  <xacro:leg_right leg_name="leg6" parent="base_link" pos_x="-0.15903" pos_y="-0.15038" pos_z="-0.03" roll="0" pitch="0" yaw="-2.384143643587"/>
+  <xacro:include filename="$(find elkapod_description)/urdf/imu.xacro" />
+  <!-- ros2_control -->
+  <xacro:include filename="$(find elkapod_description)/urdf/ros2_control.xacro" />
 </robot>

Commit message: Updated main body in URDF description, started working on inverse kinematics implementation in C++

File: elkapod_description/urdf/body/body.urdf.xacro (robot description, xacro)
@@ -1,27 +1,20 @@
 <?xml version="1.0" encoding="utf-8"?>
-<robot xmlns:xacro="http://ros.org/wiki/xacro">
-  <!-- BASE LINK -->
-    <link name="base_link">
-  </link>
-  <joint name="base_body_link" type="fixed">
-        <parent link="base_link"/>
-        <child link="body_link"/>
-        <origin xyz="0 0 0" rpy="0 0 0"/>
-  </joint>
-  <link
-    name="body_link">
-    <inertial>
-      <origin
-        xyz="-0.0049359 -0.00063942 -0.000739"
-        rpy="0 0 0" />
-      <mass
-        value="1.7153" />
-      <inertia
-        ixx="0.0088196"
-        ixy="3.5093E-05"
-        ixz="-1.7337E-08"
-        iyy="0.012893"
-        iyz="1.9595E-20"
-        izz="0.021385" />
+<robot
+  name="MainBodyAssembly - v2.SLDASM2">
+  <link
+    name="base_link">
+    <inertial>
+      <origin
+        xyz="-0.0015469 0.00072512 -0.0017855"
+        rpy="0 0 0" />
+      <mass
+        value="2.0043" />
+      <inertia
+        ixx="0.0094039"
+        ixy="0.00013899"
+        ixz="-4.7517E-07"
+        iyy="0.014031"
+        iyz="1.9401E-09"
+        izz="0.023053" />
     </inertial>
     <visual>
@@ -49,3 +42,427 @@
     </collision>
   </link>
+  <link
+    name="control_module">
+    <inertial>
+      <origin
+        xyz="0.004012 0.03538 -0.0033877"
+        rpy="0 0 0" />
+      <mass
+        value="0.43861" />
+      <inertia
+        ixx="0.00085006"
+        ixy="-1.6091E-05"
+        ixz="-1.9773E-06"
+        iyy="0.0021513"
+        iyz="1.4281E-05"
+        izz="0.0014553" />
+    </inertial>
+    <visual>
+      <origin
+        xyz="0 0 0"
+        rpy="0 0 0" />
+      <geometry>
+        <mesh
+          filename="package://elkapod_description/meshes/body/control_module.STL" />
+      </geometry>
+      <material
+        name="">
+        <color
+          rgba="0.75294 0.75294 0.75294 1" />
+      </material>
+    </visual>
+    <collision>
+      <origin
+        xyz="0 0 0"
+        rpy="0 0 0" />
+      <geometry>
+        <mesh
+          filename="package://elkapod_description/meshes/body/control_module.STL" />
+      </geometry>
+    </collision>
+  </link>
+  <joint
+    name="control_module_fixed"
+    type="fixed">
+    <origin
+      xyz="-0.0717000000000007 0.00900000000000004 0.033"
+      rpy="1.5707963267949 0 1.5707963267949" />
+    <parent
+      link="base_link" />
+    <child
+      link="control_module" />
+    <axis
+      xyz="0 0 0" />
+  </joint>
+  <link
+    name="lidar_base_footprint">
+    <inertial>
+      <origin
+        xyz="-0.0001901 6.2469E-07 0.027552"
+        rpy="0 0 0" />
+      <mass
+        value="0.3" />
+      <inertia
+        ixx="4.5255E-05"
+        ixy="1.0003E-10"
+        ixz="-1.6838E-08"
+        iyy="4.5067E-05"
+        iyz="1.7462E-09"
+        izz="6.1715E-05" />
+    </inertial>
+    <visual>
+      <origin
+        xyz="0 0 0"
+        rpy="0 0 0" />
+      <geometry>
+        <mesh
+          filename="package://elkapod_description/meshes/body/lidar_base_footprint.STL" />
+      </geometry>
+      <material
+        name="">
+        <color
+          rgba="0.75294 0.75294 0.75294 1" />
+      </material>
+    </visual>
+    <collision>
+      <origin
+        xyz="0 0 0"
+        rpy="0 0 0" />
+      <geometry>
+        <mesh
+          filename="package://elkapod_description/meshes/body/lidar_base_footprint.STL" />
+      </geometry>
+    </collision>
+  </link>
+  <joint
+    name="lidar_base_footprint_fixed"
+    type="fixed">
+    <origin
+      xyz="0.042 0.080917 -0.014678"
+      rpy="0 -1.309 -1.5708" />
+    <parent
+      link="control_module" />
+    <child
+      link="lidar_base_footprint" />
+    <axis
+      xyz="0 0 0" />
+  </joint>
+  <link
+    name="front_grille">
+    <inertial>
+      <origin
+        xyz="-1.2221E-17 0.00073241 -0.0031202"
+        rpy="0 0 0" />
+      <mass
+        value="0.051567" />
+      <inertia
+        ixx="2.0691E-05"
+        ixy="-6.8955E-21"
+        ixz="-3.4656E-20"
+        iyy="0.00017525"
+        iyz="4.3338E-07"
+        izz="0.00019204" />
+    </inertial>
+    <visual>
+      <origin
+        xyz="0 0 0"
+        rpy="0 0 0" />
+      <geometry>
+        <mesh
+          filename="package://elkapod_description/meshes/body/front_grille.STL" />
+      </geometry>
+      <material
+        name="">
+        <color
+          rgba="1 0.53725 0.18431 1" />
+      </material>
+    </visual>
+    <collision>
+      <origin
+        xyz="0 0 0"
+        rpy="0 0 0" />
+      <geometry>
+        <mesh
+          filename="package://elkapod_description/meshes/body/front_grille.STL" />
+      </geometry>
+    </collision>
+  </link>
+  <joint
+    name="front_grille_fixed"
+    type="fixed">
+    <origin
+      xyz="0.1623 0 0"
+      rpy="1.5708 0 1.5708" />
+    <parent
+      link="base_link" />
+    <child
+      link="front_grille" />
+    <axis
+      xyz="0 0 0" />
+  </joint>
+  <link
+    name="front_camera_link">
+    <inertial>
+      <origin
+        xyz="-0.0083255 0.00019292 0.00010122"
+        rpy="0 0 0" />
+      <mass
+        value="0.06" />
+      <inertia
+        ixx="1.5167E-05"
+        ixy="1.9821E-09"
+        ixz="-4.6829E-09"
+        iyy="1.558E-06"
+        iyz="1.4555E-08"
+        izz="1.3954E-05" />
+    </inertial>
+    <visual>
+      <origin
+        xyz="0 0 0"
+        rpy="0 0 0" />
+      <geometry>
+        <mesh
+          filename="package://elkapod_description/meshes/body/front_camera_link.STL" />
+      </geometry>
+      <material
+        name="">
+        <color
+          rgba="0.75294 0.75294 0.75294 1" />
+      </material>
+    </visual>
+    <collision>
+      <origin
+        xyz="0 0 0"
+        rpy="0 0 0" />
+      <geometry>
+        <mesh
+          filename="package://elkapod_description/meshes/body/front_camera_link.STL" />
+      </geometry>
+    </collision>
+  </link>
+  <joint
+    name="front_camera_link_fixed"
+    type="fixed">
+    <origin
+      xyz="0 0 0"
+      rpy="1.5707963267949 -1.5707963267949 0" />
+    <parent
+      link="front_grille" />
+    <child
+      link="front_camera_link" />
+    <axis
+      xyz="0 0 0" />
+  </joint>
+  <link
+    name="back_grilles">
+    <inertial>
+      <origin
+        xyz="0.058453 0.03 0.0029846"
+        rpy="0 0 0" />
+      <mass
+        value="0.042927" />
+      <inertia
+        ixx="1.6075E-05"
+        ixy="1.7888E-19"
+        ixz="1.0449E-08"
+        iyy="1.0788E-05"
+        iyz="4.1841E-20"
+        izz="2.593E-05" />
+    </inertial>
+    <visual>
+      <origin
+        xyz="0 0 0"
+        rpy="0 0 0" />
+      <geometry>
+        <mesh
+          filename="package://elkapod_description/meshes/body/back_grilles.STL" />
+      </geometry>
+      <material
+        name="">
+        <color
+          rgba="1 0.53725 0.18431 1" />
+      </material>
+    </visual>
+    <collision>
+      <origin
+        xyz="0 0 0"
+        rpy="0 0 0" />
+      <geometry>
+        <mesh
+          filename="package://elkapod_description/meshes/body/back_grilles.STL" />
+      </geometry>
+    </collision>
+  </link>
+  <joint
+    name="back_grilles_fixed"
+    type="fixed">
+    <origin
+      xyz="-0.15412 0.059195 -0.03"
+      rpy="1.5708 0 -1.5708" />
+    <parent
+      link="base_link" />
+    <child
+      link="back_grilles" />
+    <axis
+      xyz="0 0 0" />
+  </joint>
+  <link
+    name="left_side_grille">
+    <inertial>
+      <origin
+        xyz="0.07377 0.03 -0.037189"
+        rpy="0 0 0" />
+      <mass
+        value="0.016676" />
+      <inertia
+        ixx="1.8158E-05"
+        ixy="4.5854E-21"
+        ixz="-2.8456E-19"
+        iyy="1.1749E-05"
+        iyz="3.0718E-12"
+        izz="6.6615E-06" />
+    </inertial>
+    <visual>
+      <origin
+        xyz="0 0 0"
+        rpy="0 0 0" />
+      <geometry>
+        <mesh
+          filename="package://elkapod_description/meshes/body/left_side_grille.STL" />
+      </geometry>
+      <material
+        name="">
+        <color
+          rgba="0.25098 0.25098 0.25098 1" />
+      </material>
+    </visual>
+    <collision>
+      <origin
+        xyz="0 0 0"
+        rpy="0 0 0" />
+      <geometry>
+        <mesh
+          filename="package://elkapod_description/meshes/body/left_side_grille.STL" />
+      </geometry>
+    </collision>
+  </link>
+  <joint
+    name="left_side_grille_fixed"
+    type="fixed">
+    <origin
+      xyz="0.039489 0.19711 0.03"
+      rpy="-1.5708 0 -1.5708" />
+    <parent
+      link="base_link" />
+    <child
+      link="left_side_grille" />
+    <axis
+      xyz="0 0 0" />
+  </joint>
+  <link
+    name="right_side_grille">
+    <inertial>
+      <origin
+        xyz="0.07377 0.03 -0.037189"
+        rpy="0 0 0" />
+      <mass
+        value="0.016676" />
+      <inertia
+        ixx="1.8158E-05"
+        ixy="-4.8096E-22"
+        ixz="1.1647E-21"
+        iyy="1.1749E-05"
+        iyz="3.0718E-12"
+        izz="6.6615E-06" />
+    </inertial>
+    <visual>
+      <origin
+        xyz="0 0 0"
+        rpy="0 0 0" />
+      <geometry>
+        <mesh
+          filename="package://elkapod_description/meshes/body/right_side_grille.STL" />
+      </geometry>
+      <material
+        name="">
+        <color
+          rgba="0.25098 0.25098 0.25098 1" />
+      </material>
+    </visual>
+    <collision>
+      <origin
+        xyz="0 0 0"
+        rpy="0 0 0" />
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