Commit message: (#12) New Elkapod model for simulation, started working on robot control

File: elkapod_description/urdf/body/body.urdf.xacro (robot description, xacro)
@@ -1,312 +1,189 @@
 <?xml version="1.0" encoding="utf-8"?>
-<robot
-  name="MainBodyAssembly - v2.SLDASM2">
-  <link
-    name="base_link">
+<robot xmlns:xacro="http://ros.org/wiki/xacro">
+  <link name="base_link"/>
+  <joint name="base_body_link" type="fixed">
+        <parent link="base_link"/>
+        <child link="body_link"/>
+        <origin xyz="0 0 0" rpy="0 0 0"/>
+  </joint>
+  <link name="body_link">
     <inertial>
       <origin
         xyz="-0.0015469 0.00072512 -0.0017855"
         rpy="0 0 0" />
-      <mass
-        value="2.0043" />
-      <inertia
-        ixx="0.0094039"
-        ixy="0.00013899"
-        ixz="-4.7517E-07"
-        iyy="0.014031"
-        iyz="1.9401E-09"
-        izz="0.023053" />
-    </inertial>
-    <visual>
-      <origin
-        xyz="0 0 0"
-        rpy="0 0 0" />
-      <geometry>
-        <mesh
-          filename="package://elkapod_description/meshes/body/base_link.STL" />
-      </geometry>
-      <material
-        name="">
-        <color
-          rgba="0.8902 0.8902 0.91373 1" />
-      </material>
-    </visual>
-    <collision>
-      <origin
-        xyz="0 0 0"
-        rpy="0 0 0" />
-      <geometry>
-        <mesh
-          filename="package://elkapod_description/meshes/body/base_link.STL" />
-      </geometry>
-    </collision>
-  </link>
-  <link
-    name="control_module">
-    <inertial>
-      <origin
-        xyz="0.004012 0.03538 -0.0033877"
-        rpy="0 0 0" />
-      <mass
-        value="0.43861" />
-      <inertia
-        ixx="0.00085006"
-        ixy="-1.6091E-05"
-        ixz="-1.9773E-06"
-        iyy="0.0021513"
-        iyz="1.4281E-05"
-        izz="0.0014553" />
-    </inertial>
-    <visual>
-      <origin
-        xyz="0 0 0"
-        rpy="0 0 0" />
-      <geometry>
-        <mesh
-          filename="package://elkapod_description/meshes/body/control_module.STL" />
-      </geometry>
-      <material
-        name="">
-        <color
-          rgba="0.75294 0.75294 0.75294 1" />
-      </material>
-    </visual>
-    <collision>
-      <origin
-        xyz="0 0 0"
-        rpy="0 0 0" />
-      <geometry>
-        <mesh
-          filename="package://elkapod_description/meshes/body/control_module.STL" />
-      </geometry>
-    </collision>
-  </link>
-  <joint
-    name="control_module_fixed"
-    type="fixed">
-    <origin
-      xyz="-0.0717000000000007 0.00900000000000004 0.033"
-      rpy="1.5707963267949 0 1.5707963267949" />
-    <parent
-      link="base_link" />
-    <child
-      link="control_module" />
-    <axis
-      xyz="0 0 0" />
-  </joint>
-  <link
-    name="lidar_base_footprint">
-    <inertial>
-      <origin
-        xyz="-0.0001901 6.2469E-07 0.027552"
-        rpy="0 0 0" />
-      <mass
-        value="0.3" />
-      <inertia
-        ixx="4.5255E-05"
-        ixy="1.0003E-10"
-        ixz="-1.6838E-08"
-        iyy="4.5067E-05"
-        iyz="1.7462E-09"
-        izz="6.1715E-05" />
-    </inertial>
-    <visual>
-      <origin
-        xyz="0 0 0"
-        rpy="0 0 0" />
-      <geometry>
-        <mesh
-          filename="package://elkapod_description/meshes/body/lidar_base_footprint.STL" />
-      </geometry>
-      <material
-        name="">
-        <color
-          rgba="0.75294 0.75294 0.75294 1" />
-      </material>
-    </visual>
-    <collision>
-      <origin
-        xyz="0 0 0"
-        rpy="0 0 0" />
-      <geometry>
-        <mesh
-          filename="package://elkapod_description/meshes/body/lidar_base_footprint.STL" />
-      </geometry>
-    </collision>
-  </link>
-  <joint
-    name="lidar_base_footprint_fixed"
-    type="fixed">
-    <origin
-      xyz="0.042 0.080917 -0.014678"
-      rpy="0 -1.309 -1.5708" />
-    <parent
-      link="control_module" />
-    <child
-      link="lidar_base_footprint" />
-    <axis
-      xyz="0 0 0" />
-  </joint>
-  <link
-    name="front_grille">
-    <inertial>
-      <origin
-        xyz="-1.2221E-17 0.00073241 -0.0031202"
-        rpy="0 0 0" />
-      <mass
-        value="0.051567" />
-      <inertia
-        ixx="2.0691E-05"
-        ixy="-6.8955E-21"
-        ixz="-3.4656E-20"
-        iyy="0.00017525"
-        iyz="4.3338E-07"
-        izz="0.00019204" />
-    </inertial>
-    <visual>
-      <origin
-        xyz="0 0 0"
-        rpy="0 0 0" />
-      <geometry>
-        <mesh
-          filename="package://elkapod_description/meshes/body/front_grille.STL" />
-      </geometry>
-      <material
-        name="">
-        <color
-          rgba="1 0.53725 0.18431 1" />
-      </material>
-    </visual>
-    <collision>
-      <origin
-        xyz="0 0 0"
-        rpy="0 0 0" />
-      <geometry>
-        <mesh
-          filename="package://elkapod_description/meshes/body/front_grille.STL" />
-      </geometry>
-    </collision>
-  </link>
-  <joint
-    name="front_grille_fixed"
-    type="fixed">
-    <origin
-      xyz="0.1623 0 0"
-      rpy="1.5708 0 1.5708" />
-    <parent
-      link="base_link" />
-    <child
-      link="front_grille" />
-    <axis
-      xyz="0 0 0" />
-  </joint>
-  <link
-    name="front_camera_link">
-    <inertial>
-      <origin
-        xyz="-0.0083255 0.00019292 0.00010122"
-        rpy="0 0 0" />
-      <mass
-        value="0.06" />
-      <inertia
-        ixx="1.5167E-05"
-        ixy="1.9821E-09"
-        ixz="-4.6829E-09"
-        iyy="1.558E-06"
-        iyz="1.4555E-08"
-        izz="1.3954E-05" />
-    </inertial>
-    <visual>
-      <origin
-        xyz="0 0 0"
-        rpy="0 0 0" />
-      <geometry>
-        <mesh
-          filename="package://elkapod_description/meshes/body/front_camera_link.STL" />
-      </geometry>
-      <material
-        name="">
-        <color
-          rgba="0.75294 0.75294 0.75294 1" />
-      </material>
-    </visual>
-    <collision>
-      <origin
-        xyz="0 0 0"
-        rpy="0 0 0" />
-      <geometry>
-        <mesh
-          filename="package://elkapod_description/meshes/body/front_camera_link.STL" />
-      </geometry>
-    </collision>
-  </link>
-  <joint
-    name="front_camera_link_fixed"
-    type="fixed">
-    <origin
-      xyz="0 0 0"
-      rpy="1.5707963267949 -1.5707963267949 0" />
-    <parent
-      link="front_grille" />
-    <child
-      link="front_camera_link" />
-    <axis
-      xyz="0 0 0" />
-  </joint>
-  <link
-    name="back_grilles">
-    <inertial>
-      <origin
-        xyz="0.058453 0.03 0.0029846"
-        rpy="0 0 0" />
-      <mass
-        value="0.042927" />
-      <inertia
-        ixx="1.6075E-05"
-        ixy="1.7888E-19"
-        ixz="1.0449E-08"
-        iyy="1.0788E-05"
-        iyz="4.1841E-20"
-        izz="2.593E-05" />
-    </inertial>
-    <visual>
-      <origin
-        xyz="0 0 0"
-        rpy="0 0 0" />
-      <geometry>
-        <mesh
-          filename="package://elkapod_description/meshes/body/back_grilles.STL" />
-      </geometry>
-      <material
-        name="">
-        <color
-          rgba="1 0.53725 0.18431 1" />
-      </material>
-    </visual>
-    <collision>
-      <origin
-        xyz="0 0 0"
-        rpy="0 0 0" />
-      <geometry>
-        <mesh
-          filename="package://elkapod_description/meshes/body/back_grilles.STL" />
-      </geometry>
-    </collision>
-  </link>
-  <joint
-    name="back_grilles_fixed"
-    type="fixed">
-    <origin
-      xyz="-0.15412 0.059195 -0.03"
-      rpy="1.5708 0 -1.5708" />
-    <parent
-      link="base_link" />
-    <child
-      link="back_grilles" />
-    <axis
-      xyz="0 0 0" />
-  </joint>
-  <link
-    name="left_side_grille">
+      <mass value="2.0043" />
+      <inertia ixx="0.0094039" ixy="0.00013899" ixz="-4.7517E-07" iyy="0.014031" iyz="1.9401E-09" izz="0.023053" />
+    </inertial>
+    <visual>
+      <origin xyz="0 0 0" rpy="0 0 0" />
+      <geometry>
+        <mesh filename="package://elkapod_description/meshes/body/base_link.STL" />
+      </geometry>
+      <material name="aluminium_base"/>
+    </visual>
+    <collision>
+      <origin xyz="0 0 0" rpy="0 0 0" />
+      <geometry>
+        <mesh filename="package://elkapod_description/meshes/body/base_link.STL" />
+      </geometry>
+    </collision>
+  </link>
+  <link name="control_module">
+    <inertial>
+      <origin xyz="0.004012 0.03538 -0.0033877" rpy="0 0 0" />
+      <mass value="0.43861" />
+      <inertia ixx="0.00085006" ixy="-1.6091E-05" ixz="-1.9773E-06" iyy="0.0021513" iyz="1.4281E-05" izz="0.0014553" />
+    </inertial>
+    <visual>
+      <origin xyz="0 0 0" rpy="0 0 0" />
+      <geometry>
+        <mesh filename="package://elkapod_description/meshes/body/control_module.STL" />
+      </geometry>
+      <material name="orange_pla"/>
+    </visual>
+    <collision>
+      <origin xyz="0 0 0" rpy="0 0 0" />
+      <geometry>
+        <mesh filename="package://elkapod_description/meshes/body/control_module.STL" />
+      </geometry>
+    </collision>
+  </link>
+  <joint name="control_module_fixed" type="fixed">
+    <origin xyz="-0.0717 0.0090 0.033" rpy="1.5707963267949 0 1.5707963267949" />
+    <parent link="base_link" />
+    <child link="control_module" />
+    <axis xyz="0 0 0" />
+  </joint>
+  <link name="lidar_base_footprint">
+    <inertial>
+      <origin xyz="-0.0001901 6.2469E-07 0.027552" rpy="0 0 0" />
+      <mass value="0.3" />
+      <inertia ixx="4.5255E-05" ixy="1.0003E-10" ixz="-1.6838E-08" iyy="4.5067E-05" iyz="1.7462E-09" izz="6.1715E-05" />
+    </inertial>
+    <visual>
+      <origin xyz="0 0 0" rpy="0 0 0" />
+      <geometry>
+        <mesh filename="package://elkapod_description/meshes/body/lidar_base_footprint.STL" />
+      </geometry>
+      <material name="lidar_black"/>
+    </visual>
+    <collision>
+      <origin xyz="0 0 0" rpy="0 0 0" />
+      <geometry>
+        <mesh filename="package://elkapod_description/meshes/body/lidar_base_footprint.STL" />
+      </geometry>
+    </collision>
+  </link>
+  <joint name="lidar_base_footprint_fixed" type="fixed">
+    <origin xyz="0.042 0.080917 -0.014678" rpy="0 -1.309 -1.5708" />
+    <parent link="control_module" />
+    <child link="lidar_base_footprint" />
+    <axis xyz="0 0 0" />
+  </joint>
+  <link name="front_grille">
+    <inertial>
+      <origin xyz="-1.2221E-17 0.00073241 -0.0031202" rpy="0 0 0" />
+      <mass value="0.051567" />
+      <inertia ixx="2.0691E-05" ixy="-6.8955E-21" ixz="-3.4656E-20" iyy="0.00017525" iyz="4.3338E-07" izz="0.00019204" />
+    </inertial>
+    <visual>
+      <origin xyz="0 0 0" rpy="0 0 0" />
+      <geometry>
+        <mesh filename="package://elkapod_description/meshes/body/front_grille.STL" />
+      </geometry>
+      <material name="orange_pla"/>
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
File: elkapod_description/urdf/elkapod.urdf.xacro (robot description, xacro)
@@ -6,4 +6,6 @@
   <xacro:property name="use_sim_time" default="$(arg use_sim_time)"/>
   <!-- INCLUDES -->
+  <!-- Colors -->
+  <xacro:include filename="$(find elkapod_description)/urdf/colors.urdf.xacro" />
   <!-- Base -->
   <xacro:include filename="$(find elkapod_description)/urdf/body/body.urdf.xacro" />

File: elkapod_description/urdf/imu.xacro (robot description, xacro)
@@ -2,14 +2,4 @@
 <robot xmlns:xacro="http://www.ros.org/wiki/xacro">
     <link name="imu_link">
-        <inertial>
-            <mass value="0.01"/>
-            <origin xyz="0 0 0" rpy="0 0 0"/>
-            <inertia ixx="0.00001" ixy="0" ixz="0" iyy="0.00001" iyz="0" izz="0.00001"/>
-        </inertial>
-        <visual>
-            <geometry>
-                <sphere radius="0.02"/>
-            </geometry>
-        </visual>
     </link>
     <gazebo>

File: elkapod_description/urdf/left_leg/left_leg.urdf.xacro (robot description, xacro)
@@ -5,17 +5,8 @@
     <link name="${leg_name}_base_link">
       <inertial>
-        <origin
-          xyz="-0.00966842245121491 0.00138280482572167 0.021949062103167"
-          rpy="0 0 0" />
-        <mass
-          value="0.0812294220882115" />
-        <inertia
-          ixx="1.27671065778251E-05"
-          ixy="5.30871182380821E-13"
-          ixz="-2.82406806420912E-08"
-          iyy="2.30006815785064E-05"
-          iyz="-4.3969876504666E-07"
-          izz="1.62921012676759E-05" />
-        </inertial>
+        <origin xyz="-0.0097901 0.0013901 0.021894" rpy="0 0 0" />
+        <mass value="0.080802" />
+        <inertia ixx="1.2766E-05" ixy="5.3087E-13" ixz="-2.8241E-08" iyy="2.2999E-05" iyz="-4.397E-07" izz="1.6289E-05" />
+      </inertial>
       <visual>
         <origin xyz="0 0 0" rpy="0 0 0" />
@@ -23,7 +14,5 @@
           <mesh filename="package://elkapod_description/meshes/left_leg/base_link.STL" />
         </geometry>
-        <material name="">
-          <color rgba="0.898 0.918 0.929 1" />
-        </material>
+        <material name="leg_black"/>
       </visual>
       <collision>
@@ -43,7 +32,7 @@
     <link name="${leg_name}_linkA">
       <inertial>
-        <origin xyz="0.03385 0.00126 0.00129" rpy="0 0 0" />
-        <mass value="0.04544" />
-        <inertia ixx="1.9828E-05" ixy="1.195E-12" ixz="-5.464E-13" iyy="1.6727E-05" iyz="-1.074E-12" izz="1.6727E-05" />
+        <origin xyz="0.033799 0.00051236 0.00054959" rpy="0 0 0" />
+        <mass value="0.042693" />
+        <inertia ixx="1.9802E-05" ixy="8.7559E-13" ixz="-5.8218E-13" iyy="1.6706E-05" iyz="-1.8291E-12" izz="1.6706E-05" />
       </inertial>
       <visual>
@@ -52,7 +41,5 @@
           <mesh filename="package://elkapod_description/meshes/left_leg/linkA.STL" />
         </geometry>
-        <material name="">
-          <color rgba="0.898 0.918 0.929 1" />
-        </material>
+        <material name="leg_black"/>
       </visual>
       <collision>
@@ -74,7 +61,7 @@
     <link name="${leg_name}_linkB">
       <inertial>
-        <origin xyz="0.0318 0.03385 0.00347" rpy="0 0 0" />
-        <mass value="0.17153" />
-        <inertia ixx="3.545E-05" ixy="-8.639E-06" ixz="-4.662E-07" iyy="3.792E-05" iyz="5.374E-07" izz="3.388E-05" />
+        <origin xyz="0.046185 0.0047076 0.0034661" rpy="0 0 0" />
+        <mass value="0.16871" />
+        <inertia ixx="2.7946E-05" ixy="-8.4625E-13" ixz="2.1218E-12" iyy="4.5398E-05" iyz="7.1144E-07" izz="3.3864E-05" />
       </inertial>
       <visual>
@@ -83,7 +70,5 @@
           <mesh filename="package://elkapod_description/meshes/left_leg/linkB.STL" />
         </geometry>
-        <material name="">
-          <color rgba="0.251 0.251 0.251 1" />
-        </material>
+        <material name="leg_black"/>
       </visual>
       <collision>
@@ -96,5 +81,5 @@
     <!-- Joint J2 -->
     <joint name="${leg_name}_J2" type="revolute">
-      <origin xyz="0.0676 0 0" rpy="1.5708 0.7146 0" />
+      <origin xyz="0.0676 0 0" rpy="1.5708 0 0" />
       <parent link="${leg_name}_linkA" />
       <child link="${leg_name}_linkB" />
@@ -105,7 +90,7 @@
     <link name="${leg_name}_linkC">
       <inertial>
-        <origin xyz="0.03063 -0.05443 -0.00114" rpy="0 0 0" />
-        <mass value="0.04744" />
-        <inertia ixx="5.613E-05" ixy="1.497E-05" ixz="1.598E-07" iyy="2.328E-05" iyz="-2.931E-07" izz="5.235E-05" />
+        <origin xyz="0.062526 0.013836 -0.00039598" rpy="0 0 0" />
+        <mass value="0.045919" />
+        <inertia ixx="1.7731E-05" ixy="-3.3492E-06" ixz="3.2696E-07" iyy="6.1677E-05" iyz="6.793E-08" izz="5.2343E-05" />
       </inertial>
       <visual>
@@ -114,7 +99,5 @@
           <mesh filename="package://elkapod_description/meshes/left_leg/linkC.STL" />
         </geometry>
-        <material name="">
-          <color rgba="1 0.529 0 1" />
-        </material>
+        <material name="orange_pla"/>
       </visual>
       <collision>
@@ -127,5 +110,5 @@
     <!-- Joint J3 -->
     <joint name="${leg_name}_J3" type="revolute">
-      <origin xyz="0.06977 0.06053 0" rpy="0 0 1.951" />
+      <origin xyz="0.0923692721756408 0 0" rpy="0 0 0" />
       <parent link="${leg_name}_linkB" />
       <child link="${leg_name}_linkC" />
@@ -136,7 +119,7 @@
     <link name="${leg_name}_FCP">
       <inertial>
-        <origin xyz="0.00034 0 0" rpy="0 0 0" />
-        <mass value="0.01116" />
-        <inertia ixx="1.199E-06" ixy="3.584E-24" ixz="-1.195E-23" iyy="1.067E-06" iyz="-7.636E-37" izz="1.067E-06" />
+        <origin xyz="0.000341547110339208 2.77555756156289E-17 1.73472347597681E-18" rpy="0 0 0" />
+        <mass value="0.0111617991818567" />
+        <inertia ixx="1.19862E-06" ixy="-5.67881E-40" ixz="-4.86711E-24" iyy="1.06703E-06" iyz="-1.94856E-26" izz="1.06703E-06" />
       </inertial>
       <visual>
@@ -146,5 +129,5 @@
         </geometry>
         <material name="">
-          <color rgba="0.298 0.298 0.298 1" />
+          <color rgba="1 0 0 1" />
         </material>
       </visual>
@@ -158,5 +141,5 @@
     <!-- Fixed Joint for FCP -->
     <joint name="${leg_name}_FCP_joint" type="fixed">
-      <origin xyz="0.07008 -0.20186 0" rpy="0 0 -1.571" />
+      <origin xyz="0.2135 0.0085747 0" rpy="0 0 -0.29403" />
       <parent link="${leg_name}_linkC" />
       <child link="${leg_name}_FCP" />
