Commit message: (#12) New Elkapod model for simulation, started working on robot control

File: elkapod_description/urdf/right_leg/right_leg.urdf.xacro (robot description, xacro)
@@ -4,24 +4,22 @@
     <!-- Base link -->
     <link name="${leg_name}_base_link">
-        <inertial>
-            <origin xyz="-0.0096684 -0.0013828 0.021949" rpy="0 0 0" />
-            <mass value="0.081229" />
-            <inertia ixx="1.2767E-05" ixy="5.1064E-13" ixz="-2.8243E-08" iyy="2.3001E-05" iyz="4.397E-07" izz="1.6292E-05" />
-        </inertial>
-        <visual>
-            <origin xyz="0 0 0" rpy="0 0 0" />
-            <geometry>
-                <mesh filename="package://elkapod_description/meshes/right_leg/base_link.STL" />
-            </geometry>
-            <material name="">
-                <color rgba="0.69804 0.69804 0.69804 1" />
-            </material>
-        </visual>
-        <collision>
-            <origin xyz="0 0 0" rpy="0 0 0" />
-            <geometry>
-                <mesh filename="package://elkapod_description/meshes/right_leg/base_link.STL" />
-            </geometry>
-        </collision>
+      <inertial>
+        <origin xyz="-0.00979014713716649 -0.00139011782449186 0.0218935307853371" rpy="0 0 0" />
+        <mass value="0.0808021222974834" />
+        <inertia ixx="1.27655E-05" ixy="5.10643E-13" ixz="-2.82428E-08" iyy="2.29991E-05" iyz="4.39699E-07" izz="1.62889E-05" />
+      </inertial>
+      <visual>
+        <origin xyz="0 0 0" rpy="0 0 0" />
+        <geometry>
+          <mesh filename="package://elkapod_description/meshes/right_leg/base_link.STL" />
+        </geometry>
+        <material name="leg_black"/>
+      </visual>
+      <collision>
+        <origin xyz="0 0 0" rpy="0 0 0" />
+        <geometry>
+          <mesh filename="package://elkapod_description/meshes/right_leg/base_link.STL" />
+        </geometry>
+      </collision>
     </link>
     <joint name="${leg_name}_base_joint" type="fixed">
@@ -33,24 +31,22 @@
     <!-- Link A -->
     <link name="${leg_name}_linkA">
-        <inertial>
-            <origin xyz="0.033735 -0.0012826 0.0013134" rpy="0 0 0" />
-            <mass value="0.045199" />
-            <inertia ixx="1.9826E-05" ixy="-2.3136E-13" ixz="-5.4127E-13" iyy="1.6726E-05" iyz="-2.1687E-12" izz="1.6726E-05" />
-        </inertial>
-        <visual>
-            <origin xyz="0 0 0" rpy="0 0 0" />
-            <geometry>
-                <mesh filename="package://elkapod_description/meshes/right_leg/linkA.STL" />
-            </geometry>
-            <material name="">
-                <color rgba="0.898039215686275 0.917647058823529 0.929411764705882 1" />
-            </material>
-        </visual>
-        <collision>
-            <origin xyz="0 0 0" rpy="0 0 0" />
-            <geometry>
-                <mesh filename="package://elkapod_description/meshes/right_leg/linkA.STL" />
-            </geometry>
-        </collision>
+      <inertial>
+        <origin xyz="0.0337988193565861 -0.000554586093327376 0.000549586085186449" rpy="0 0 0" />
+        <mass value="0.0426933486153037" />
+        <inertia ixx="1.98022E-05" ixy="-2.13458E-13" ixz="-5.41372E-13" iyy="1.670609E-05" iyz="-2.17248E-12" izz="1.67061E-05" />
+      </inertial>
+      <visual>
+        <origin xyz="0 0 0" rpy="0 0 0" />
+        <geometry>
+          <mesh filename="package://elkapod_description/meshes/right_leg/linkA.STL" />
+        </geometry>
+        <material name="leg_black"/>
+      </visual>
+      <collision>
+        <origin xyz="0 0 0" rpy="0 0 0" />
+        <geometry>
+          <mesh filename="package://elkapod_description/meshes/right_leg/linkA.STL" />
+        </geometry>
+      </collision>
     </link>
     <!-- Joint J1 -->
@@ -64,24 +60,22 @@
     <!-- Link B -->
     <link name="${leg_name}_linkB">
-        <inertial>
-            <origin xyz="0.046253 0.0040276 -0.0026292" rpy="0 0 0" />
-            <mass value="0.1717" />
-            <inertia ixx="2.7961E-05" ixy="2.7244E-07" ixz="-1.1105E-08" iyy="4.5406E-05" iyz="-7.1135E-07" izz="3.3884E-05" />
-        </inertial>
-        <visual>
-            <origin xyz="0 0 0" rpy="0 0 0" />
-            <geometry>
-                <mesh filename="package://elkapod_description/meshes/right_leg/linkB.STL" />
-            </geometry>
-            <material name="">
-                <color rgba="0.250980392156863 0.250980392156863 0.250980392156863 1" />
-            </material>
-        </visual>
-        <collision>
-            <origin xyz="0 0 0" rpy="0 0 0" />
-            <geometry>
-                <mesh filename="package://elkapod_description/meshes/right_leg/linkB.STL" />
-            </geometry>
-        </collision>
+      <inertial>
+        <origin xyz="0.0461949754482681 0.00470912944794107 -0.00261992673183065" rpy="0 0 0" />
+        <mass value="0.168678406706635" />
+        <inertia ixx="2.79458E-05" ixy="8.13719E-13" ixz="2.16502E-12" iyy="4.53975E-05" iyz="-7.11437E-07" izz="3.38637E-05" />
+      </inertial>
+      <visual>
+        <origin xyz="0 0 0" rpy="0 0 0" />
+        <geometry>
+          <mesh filename="package://elkapod_description/meshes/right_leg/linkB.STL" />
+        </geometry>
+        <material name="leg_black"/>
+      </visual>
+      <collision>
+        <origin xyz="0 0 0" rpy="0 0 0" />
+        <geometry>
+          <mesh filename="package://elkapod_description/meshes/right_leg/linkB.STL" />
+        </geometry>
+      </collision>
     </link>
     <!-- Joint J2 -->
@@ -95,28 +89,26 @@
     <!-- Link C -->
     <link name="${leg_name}_linkC">
-        <inertial>
-            <origin xyz="0.030676 -0.054506 0.0011426" rpy="0 0 0" />
-            <mass value="0.04737" />
-            <inertia ixx="5.613E-05" ixy="1.4973E-05" ixz="1.5976E-07" iyy="2.3284E-05" iyz="-2.9313E-07" izz="5.2352E-05" />
-        </inertial>
-        <visual>
-            <origin xyz="0 0 0" rpy="0 0 0" />
-            <geometry>
-                <mesh filename="package://elkapod_description/meshes/right_leg/linkC.STL" />
-            </geometry>
-            <material name="">
-                <color rgba="1 0.529411764705882 0 1" />
-            </material>
-        </visual>
-        <collision>
-            <origin xyz="0 0 0" rpy="0 0 0" />
-            <geometry>
-                <mesh filename="package://elkapod_description/meshes/right_leg/linkC.STL" />
-            </geometry>
-        </collision>
+      <inertial>
+        <origin xyz="0.0626878415018562 0.0138717503264788 0.00052553418423365" rpy="0 0 0" />
+        <mass value="0.0457999682692435" />
+        <inertia ixx="1.77293E-05" ixy="-3.34917E-06" ixz="3.26962E-07" iyy="6.16756E-05" iyz="6.79304E-08" izz="5.23429E-05" />
+      </inertial>
+      <visual>
+        <origin xyz="0 0 0" rpy="0 0 0" />
+        <geometry>
+          <mesh filename="package://elkapod_description/meshes/right_leg/linkC.STL" />
+        </geometry>
+        <material name="orange_pla"/>
+      </visual>
+      <collision>
+        <origin xyz="0 0 0" rpy="0 0 0" />
+        <geometry>
+          <mesh filename="package://elkapod_description/meshes/right_leg/linkC.STL" />
+        </geometry>
+      </collision>
     </link>
     <!-- Joint J3 -->
     <joint name="${leg_name}_J3" type="revolute">
-        <origin xyz="0.092358 -0.0014421 0" rpy="0 0 1.2435" />
+        <origin xyz="0.092358 -0.0014421 0" rpy="0 0 0" />
         <parent link="${leg_name}_linkB" />
         <child link="${leg_name}_linkC" />
@@ -126,28 +118,28 @@
     <!-- FCP link -->
     <link name="${leg_name}_FCP">
-        <inertial>
-            <origin xyz="0.0003415 8.3267E-17 6.9389E-18" rpy="0 0 0" />
-            <mass value="0.011162" />
-            <inertia ixx="1.1986E-06" ixy="-7.1946E-23" ixz="-5.5609E-24" iyy="1.067E-06" iyz="4.1316E-36" izz="1.067E-06" />
-        </inertial>
-        <visual>
-            <origin xyz="0 0 0" rpy="0 0 0" />
-            <geometry>
-                <mesh filename="package://elkapod_description/meshes/right_leg/FCP.STL" />
-            </geometry>
-            <material name="">
-                <color rgba="0.298039215686275 0.298039215686275 0.298039215686275 1" />
-            </material>
-        </visual>
-        <collision>
-            <origin xyz="0 0 0" rpy="0 0 0" />
-            <geometry>
-                <mesh filename="package://elkapod_description/meshes/right_leg/FCP.STL" />
-            </geometry>
-        </collision>
+      <inertial>
+        <origin xyz="0.000341547110338625 4.16333634234434E-17 -3.46944695195361E-17" rpy="0 0 0" />
+        <mass value="0.0111617991818567" />
+        <inertia ixx="1.19862E-06" ixy="1.05879E-22" ixz="1.15499E-24" iyy="1.06703E-06" iyz="9.44775E-26" izz="1.06703E-06" />
+      </inertial>
+      <visual>
+        <origin xyz="0 0 0" rpy="0 0 0" />
+        <geometry>
+          <mesh filename="package://elkapod_description/meshes/right_leg/FCP.STL" />
+        </geometry>
+        <material name="">
+          <color rgba="1 0 0 1" />
+        </material>
+      </visual>
+      <collision>
+        <origin xyz="0 0 0" rpy="0 0 0" />
+        <geometry>
+          <mesh filename="package://elkapod_description/meshes/right_leg/FCP.STL" />
+        </geometry>
+      </collision>
     </link>
     <!-- Fixed joint for FCP -->
     <joint name="${leg_name}_FCP_joint" type="fixed">
-        <origin xyz="0.070083 -0.20186 0" rpy="0 0 -1.5708" />
+        <origin xyz="0.213503787197785 0.00857470533092818 0" rpy="0 0 -0.294032099334707" />
         <parent link="${leg_name}_linkC" />
         <child link="${leg_name}_FCP" />

Commit message: Modified robot description, creating working 3d lidar sensor publishing data from gazebo to ROS

File: elkapod_description/urdf/body/body.urdf.xacro (robot description, xacro)
@@ -55,30 +55,4 @@
     <axis xyz="0 0 0" />
   </joint>
-  <link name="lidar_base_footprint">
-    <inertial>
-      <origin xyz="-0.0001901 6.2469E-07 0.027552" rpy="0 0 0" />
-      <mass value="0.3" />
-      <inertia ixx="4.5255E-05" ixy="1.0003E-10" ixz="-1.6838E-08" iyy="4.5067E-05" iyz="1.7462E-09" izz="6.1715E-05" />
-    </inertial>
-    <visual>
-      <origin xyz="0 0 0" rpy="0 0 0" />
-      <geometry>
-        <mesh filename="package://elkapod_description/meshes/body/lidar_base_footprint.STL" />
-      </geometry>
-      <material name="lidar_black"/>
-    </visual>
-    <collision>
-      <origin xyz="0 0 0" rpy="0 0 0" />
-      <geometry>
-        <mesh filename="package://elkapod_description/meshes/body/lidar_base_footprint.STL" />
-      </geometry>
-    </collision>
-  </link>
-  <joint name="lidar_base_footprint_fixed" type="fixed">
-    <origin xyz="0.042 0.080917 -0.014678" rpy="0 -1.309 -1.5708" />
-    <parent link="control_module" />
-    <child link="lidar_base_footprint" />
-    <axis xyz="0 0 0" />
-  </joint>
   <link name="front_grille">
     <inertial>

File: elkapod_description/urdf/elkapod.urdf.xacro (robot description, xacro)
@@ -19,5 +19,7 @@
   <xacro:leg_right leg_name="leg4" parent="base_link" pos_x="0.0138" pos_y="-0.1643" pos_z="-0.03" roll="0" pitch="0" yaw="-1.57"/>
   <xacro:leg_right leg_name="leg6" parent="base_link" pos_x="-0.15903" pos_y="-0.15038" pos_z="-0.03" roll="0" pitch="0" yaw="-2.384143643587"/>
+  <!-- Sensors -->
   <xacro:include filename="$(find elkapod_description)/urdf/imu.xacro" />
+  <xacro:include filename="$(find elkapod_description)/urdf/lidar.xacro" />
   <!-- ros2_control -->
   <xacro:include filename="$(find elkapod_description)/urdf/ros2_control.xacro" />

Commit message: Added front rgbd camera (almost, frame issues), moved sensors to seperate directory

File: elkapod_description/urdf/body/body.urdf.xacro (robot description, xacro)
@@ -79,30 +79,4 @@
     <parent link="base_link" />
     <child link="front_grille" />
-    <axis xyz="0 0 0" />
-  </joint>
-  <link name="front_camera_link">
-    <inertial>
-      <origin xyz="-0.0083255 0.00019292 0.00010122" rpy="0 0 0" />
-      <mass value="0.06" />
-      <inertia ixx="1.5167E-05" ixy="1.9821E-09" ixz="-4.6829E-09" iyy="1.558E-06" iyz="1.4555E-08" izz="1.3954E-05" />
-    </inertial>
-    <visual>
-      <origin xyz="0 0 0" rpy="0 0 0" />
-      <geometry>
-        <mesh filename="package://elkapod_description/meshes/body/front_camera_link.STL" />
-      </geometry>
-      <material name="pure_black"/>
-    </visual>
-    <collision>
-      <origin xyz="0 0 0" rpy="0 0 0" />
-      <geometry>
-        <mesh filename="package://elkapod_description/meshes/body/front_camera_link.STL" />
-      </geometry>
-    </collision>
-  </link>
-  <joint name="front_camera_link_fixed" type="fixed">
-    <origin xyz="0 0 0" rpy="1.5707963267949 -1.5707963267949 0" />
-    <parent link="front_grille" />
-    <child link="front_camera_link" />
     <axis xyz="0 0 0" />
   </joint>

File: elkapod_description/urdf/elkapod.urdf.xacro (robot description, xacro)
@@ -20,6 +20,7 @@
   <xacro:leg_right leg_name="leg6" parent="base_link" pos_x="-0.15903" pos_y="-0.15038" pos_z="-0.03" roll="0" pitch="0" yaw="-2.384143643587"/>
   <!-- Sensors -->
-  <xacro:include filename="$(find elkapod_description)/urdf/imu.xacro" />
-  <xacro:include filename="$(find elkapod_description)/urdf/lidar.xacro" />
+  <xacro:include filename="$(find elkapod_description)/urdf/sensors/imu.xacro" />
+  <xacro:include filename="$(find elkapod_description)/urdf/sensors/lidar.xacro" />
+  <xacro:include filename="$(find elkapod_description)/urdf/sensors/depth_camera.xacro" />
   <!-- ros2_control -->
   <xacro:include filename="$(find elkapod_description)/urdf/ros2_control.xacro" />

File: elkapod_description/urdf/sensors/lidar.xacro (robot description, xacro)
@@ -28,8 +28,15 @@
         <axis xyz="0 0 0" />
     </joint>
-    <gazebo reference="lidar_base_footprint">
-        <sensor name="lidar" type="gpu_lidar">lea
+    <link name="lidar_optical"></link>
+    <joint name="lidar_base_optical_fixed" type="fixed">
+        <origin xyz="0 0 0.04534" rpy="0 0 0" />
+        <parent link="lidar_base_footprint" />
+        <child link="lidar_optical" />
+        <axis xyz="0 0 0" />
+    </joint>
+    <gazebo reference="lidar_optical">
+        <sensor name="lidar" type="gpu_lidar">
             <always_on>true</always_on>
-            <update_rate>5</update_rate>
+            <update_rate>2</update_rate>
             <visualize>true</visualize>
             <topic>lidar_data</topic>
@@ -37,5 +44,5 @@
                 <scan>
                     <horizontal>
-                        <samples>90</samples>
+                        <samples>45</samples>
                         <resolution>1</resolution>
                         <min_angle>-3.14</min_angle>
@@ -55,4 +62,5 @@
                 </range>
             </lidar>
+            <gz_frame_id>lidar_optical</gz_frame_id>
         </sensor>
     </gazebo>

Commit message: Navigation core sensors (#38)
* Modified robot description, creating working 3d lidar sensor publishing data from gazebo to ROS

* Added front rgbd camera (almost, frame issues), moved sensors to seperate directory

* Finished tuning sensor parameters

* Removed imu xacro file
Added sim macros for sensors

File: elkapod_description/urdf/body/body.urdf.xacro (robot description, xacro)
@@ -55,30 +55,4 @@
     <axis xyz="0 0 0" />
   </joint>
-  <link name="lidar_base_footprint">
-    <inertial>
-      <origin xyz="-0.0001901 6.2469E-07 0.027552" rpy="0 0 0" />
-      <mass value="0.3" />
-      <inertia ixx="4.5255E-05" ixy="1.0003E-10" ixz="-1.6838E-08" iyy="4.5067E-05" iyz="1.7462E-09" izz="6.1715E-05" />
-    </inertial>
-    <visual>
-      <origin xyz="0 0 0" rpy="0 0 0" />
-      <geometry>
-        <mesh filename="package://elkapod_description/meshes/body/lidar_base_footprint.STL" />
-      </geometry>
-      <material name="lidar_black"/>
-    </visual>
-    <collision>
-      <origin xyz="0 0 0" rpy="0 0 0" />
-      <geometry>
-        <mesh filename="package://elkapod_description/meshes/body/lidar_base_footprint.STL" />
-      </geometry>
-    </collision>
-  </link>
-  <joint name="lidar_base_footprint_fixed" type="fixed">
-    <origin xyz="0.042 0.080917 -0.014678" rpy="0 -1.309 -1.5708" />
-    <parent link="control_module" />
-    <child link="lidar_base_footprint" />
-    <axis xyz="0 0 0" />
-  </joint>
   <link name="front_grille">
     <inertial>
@@ -105,30 +79,4 @@
     <parent link="base_link" />
     <child link="front_grille" />
-    <axis xyz="0 0 0" />
-  </joint>
-  <link name="front_camera_link">
-    <inertial>
-      <origin xyz="-0.0083255 0.00019292 0.00010122" rpy="0 0 0" />
-      <mass value="0.06" />
-      <inertia ixx="1.5167E-05" ixy="1.9821E-09" ixz="-4.6829E-09" iyy="1.558E-06" iyz="1.4555E-08" izz="1.3954E-05" />
-    </inertial>
-    <visual>
-      <origin xyz="0 0 0" rpy="0 0 0" />
-      <geometry>
-        <mesh filename="package://elkapod_description/meshes/body/front_camera_link.STL" />
-      </geometry>
-      <material name="pure_black"/>
-    </visual>
-    <collision>
-      <origin xyz="0 0 0" rpy="0 0 0" />
-      <geometry>
-        <mesh filename="package://elkapod_description/meshes/body/front_camera_link.STL" />
-      </geometry>
-    </collision>
-  </link>
-  <joint name="front_camera_link_fixed" type="fixed">
-    <origin xyz="0 0 0" rpy="1.5707963267949 -1.5707963267949 0" />
-    <parent link="front_grille" />
-    <child link="front_camera_link" />
     <axis xyz="0 0 0" />
   </joint>

File: elkapod_description/urdf/elkapod.urdf.xacro (robot description, xacro)
@@ -17,4 +17,9 @@
   <xacro:leg_right leg_name="leg4" parent="base_link" pos_x="0.0138" pos_y="-0.1643" pos_z="-0.03" roll="0" pitch="0" yaw="-1.57"/>
   <xacro:leg_right leg_name="leg6" parent="base_link" pos_x="-0.15903" pos_y="-0.15038" pos_z="-0.03" roll="0" pitch="0" yaw="-2.384143643587"/>
+  <!-- Sensors -->
+  <xacro:include filename="$(find elkapod_description)/urdf/sensors/lidar.xacro" />
+  <xacro:include filename="$(find elkapod_description)/urdf/sensors/depth_camera.xacro" />
+  <xacro:elkapod_sensors_lidar sim_mode="$(arg sim_mode)"/>
+  <xacro:elkapod_sensors_fron_camera sim_mode="$(arg sim_mode)"/>
   <!-- ros2_control -->
   <xacro:include filename="$(find elkapod_description)/ros2_control/elkapod.ros2_control.xacro" />
