Commit message: #17 Corrected joint angle limits for the robot

File: elkapod_description/urdf/left_leg/left_leg.urdf.xacro (robot description, xacro)
@@ -56,5 +56,5 @@
       <child link="${leg_name}_linkA" />
       <axis xyz="0 0 1" />
-      <limit lower="-1.57" upper="1.57" effort="5" velocity="1.0" />
+      <limit lower="-1.57" upper="1.57" effort="50" velocity="7.3" />
     </joint>
     <!-- Link B -->
@@ -85,5 +85,5 @@
       <child link="${leg_name}_linkB" />
       <axis xyz="0 0 1" />
-      <limit lower="-1.57" upper="1.57" effort="5" velocity="1.0" />
+      <limit lower="-1.57" upper="1.57" effort="50" velocity="7.3" />
     </joint>
     <!-- Link C -->
@@ -114,5 +114,5 @@
       <child link="${leg_name}_linkC" />
       <axis xyz="0 0 1" />
-      <limit lower="-3.14" upper="1.57" effort="5" velocity="1.0" />
+      <limit lower="-3.14" upper="1.57" effort="50" velocity="7.3" />
     </joint>
     <!-- FCP Link -->

File: elkapod_description/urdf/right_leg/right_leg.urdf.xacro (robot description, xacro)
@@ -56,5 +56,5 @@
         <child link="${leg_name}_linkA" />
         <axis xyz="0 0 1" />
-        <limit lower="-1.57" upper="1.57" effort="5" velocity="1.0" />
+        <limit lower="-1.57" upper="1.57" effort="50" velocity="7.3" />
     </joint>
     <!-- Link B -->
@@ -85,5 +85,5 @@
         <child link="${leg_name}_linkB" />
         <axis xyz="0 0 1" />
-        <limit lower="-1.57" upper="1.57" effort="5" velocity="1.0" />
+        <limit lower="-1.57" upper="1.57" effort="50" velocity="7.3" />
     </joint>
     <!-- Link C -->
@@ -114,5 +114,5 @@
         <child link="${leg_name}_linkC" />
         <axis xyz="0 0 1" />
-        <limit lower="-3.14" upper="3.14" effort="5" velocity="1.0" />
+        <limit lower="-3.14" upper="3.14" effort="50" velocity="7.3" />
     </joint>
     <!-- FCP link -->

File: elkapod_description/urdf/ros2_control.xacro (robot description, xacro)
@@ -18,21 +18,21 @@
             </hardware>
             <xacro:joint_interface name="leg1_J1" min_pos_rad="-1.57" max_pos_rad="1.57" initial_angle_rad="0.0"/>
-            <xacro:joint_interface name="leg1_J2" min_pos_rad="-3.14" max_pos_rad="3.14" initial_angle_rad="0.0"/>
-            <xacro:joint_interface name="leg1_J3" min_pos_rad="-3.14" max_pos_rad="3.14" initial_angle_rad="0.0"/>
+            <xacro:joint_interface name="leg1_J2" min_pos_rad="-1.57" max_pos_rad="1.57" initial_angle_rad="0.0"/>
+            <xacro:joint_interface name="leg1_J3" min_pos_rad="-3.14" max_pos_rad="0.0" initial_angle_rad="0.0"/>
             <xacro:joint_interface name="leg3_J1" min_pos_rad="-1.57" max_pos_rad="1.57" initial_angle_rad="0.0"/>
-            <xacro:joint_interface name="leg3_J2" min_pos_rad="-3.14" max_pos_rad="3.14" initial_angle_rad="0.0"/>
-            <xacro:joint_interface name="leg3_J3" min_pos_rad="-3.14" max_pos_rad="3.14" initial_angle_rad="0.0"/>
+            <xacro:joint_interface name="leg3_J2" min_pos_rad="-1.57" max_pos_rad="1.57" initial_angle_rad="0.0"/>
+            <xacro:joint_interface name="leg3_J3" min_pos_rad="-3.14" max_pos_rad="0.0" initial_angle_rad="0.0"/>
             <xacro:joint_interface name="leg5_J1" min_pos_rad="-1.57" max_pos_rad="1.57" initial_angle_rad="0.0"/>
-            <xacro:joint_interface name="leg5_J2" min_pos_rad="-3.14" max_pos_rad="3.14" initial_angle_rad="0.0"/>
-            <xacro:joint_interface name="leg5_J3" min_pos_rad="-3.14" max_pos_rad="3.14" initial_angle_rad="0.0"/>
+            <xacro:joint_interface name="leg5_J2" min_pos_rad="-1.57" max_pos_rad="1.57" initial_angle_rad="0.0"/>
+            <xacro:joint_interface name="leg5_J3" min_pos_rad="-3.14" max_pos_rad="0.0" initial_angle_rad="0.0"/>
             <xacro:joint_interface name="leg2_J1" min_pos_rad="-1.57" max_pos_rad="1.57" initial_angle_rad="0.0"/>
-            <xacro:joint_interface name="leg2_J2" min_pos_rad="-3.14" max_pos_rad="3.14" initial_angle_rad="0.0"/>
-            <xacro:joint_interface name="leg2_J3" min_pos_rad="-3.14" max_pos_rad="3.14" initial_angle_rad="0.0"/>
+            <xacro:joint_interface name="leg2_J2" min_pos_rad="-1.57" max_pos_rad="1.57" initial_angle_rad="0.0"/>
+            <xacro:joint_interface name="leg2_J3" min_pos_rad="-3.14" max_pos_rad="0.0" initial_angle_rad="0.0"/>
             <xacro:joint_interface name="leg4_J1" min_pos_rad="-1.57" max_pos_rad="1.57" initial_angle_rad="0.0"/>
-            <xacro:joint_interface name="leg4_J2" min_pos_rad="-3.14" max_pos_rad="3.14" initial_angle_rad="0.0"/>
-            <xacro:joint_interface name="leg4_J3" min_pos_rad="-3.14" max_pos_rad="3.14" initial_angle_rad="0.0"/>
+            <xacro:joint_interface name="leg4_J2" min_pos_rad="-1.57" max_pos_rad="1.57" initial_angle_rad="0.0"/>
+            <xacro:joint_interface name="leg4_J3" min_pos_rad="-3.14" max_pos_rad="0.0" initial_angle_rad="0.0"/>
             <xacro:joint_interface name="leg6_J1" min_pos_rad="-1.57" max_pos_rad="1.57" initial_angle_rad="0.0"/>
-            <xacro:joint_interface name="leg6_J2" min_pos_rad="-3.14" max_pos_rad="3.14" initial_angle_rad="0.0"/>
-            <xacro:joint_interface name="leg6_J3" min_pos_rad="-3.14" max_pos_rad="3.14" initial_angle_rad="0.0"/>
+            <xacro:joint_interface name="leg6_J2" min_pos_rad="-1.57" max_pos_rad="1.57" initial_angle_rad="0.0"/>
+            <xacro:joint_interface name="leg6_J3" min_pos_rad="-3.14" max_pos_rad="0.0" initial_angle_rad="0.0"/>
         </ros2_control>
     </xacro:if>

Commit message: #17 Replaced mesh foot with geometry sphere foot thus improving simulation speed and enabling friction

File: elkapod_description/urdf/left_leg/left_leg.urdf.xacro (robot description, xacro)
@@ -126,5 +126,5 @@
         <origin xyz="0 0 0" rpy="0 0 0" />
         <geometry>
-          <mesh filename="package://elkapod_description/meshes/left_leg/FCP.STL" />
+          <sphere radius="0.01"/>
         </geometry>
         <material name="">
@@ -135,16 +135,12 @@
         <origin xyz="0 0 0" rpy="0 0 0" />
         <geometry>
-          <mesh filename="package://elkapod_description/meshes/left_leg/FCP.STL" />
+          <sphere radius="0.01"/>
         </geometry>
-        <surface>
-          <friction>
-            <ode>
-              <mu>1000.0</mu>
-              <mu2>1000.0</mu2>
-            </ode>
-          </friction>
-        </surface>
       </collision>
     </link>
+    <gazebo reference="${leg_name}_FCP">
+      <mu1>1000.0</mu1>
+      <mu2>1000.0</mu2>
+    </gazebo>
     <!-- Fixed Joint for FCP -->
     <joint name="${leg_name}_FCP_joint" type="fixed">

File: elkapod_description/urdf/right_leg/right_leg.urdf.xacro (robot description, xacro)
@@ -126,5 +126,5 @@
         <origin xyz="0 0 0" rpy="0 0 0" />
         <geometry>
-          <mesh filename="package://elkapod_description/meshes/right_leg/FCP.STL" />
+          <sphere radius="0.01"/>
         </geometry>
         <material name="">
@@ -135,16 +135,12 @@
         <origin xyz="0 0 0" rpy="0 0 0" />
         <geometry>
-          <mesh filename="package://elkapod_description/meshes/right_leg/FCP.STL" />
+          <sphere radius="0.01"/>
         </geometry>
-        <surface>
-          <friction>
-            <ode>
-              <mu>1000.0</mu>
-              <mu2>1000.0</mu2>
-            </ode>
-          </friction>
-        </surface>
       </collision>
     </link>
+    <gazebo reference="${leg_name}_FCP">
+      <mu1>1000.0</mu1>
+      <mu2>1000.0</mu2>
+    </gazebo>
     <!-- Fixed joint for FCP -->
     <joint name="${leg_name}_FCP_joint" type="fixed">

Commit message: #17 Added elkapod_motion_manager to the launch file, changed effort in the joints to 3.5Nm, other minor changes

File: elkapod_description/urdf/left_leg/left_leg.urdf.xacro (robot description, xacro)
@@ -56,5 +56,5 @@
       <child link="${leg_name}_linkA" />
       <axis xyz="0 0 1" />
-      <limit lower="-1.57" upper="1.57" effort="50" velocity="7.3" />
+      <limit lower="-1.57" upper="1.57" effort="3.5" velocity="7.3" />
     </joint>
     <!-- Link B -->
@@ -85,5 +85,5 @@
       <child link="${leg_name}_linkB" />
       <axis xyz="0 0 1" />
-      <limit lower="-1.57" upper="1.57" effort="50" velocity="7.3" />
+      <limit lower="-1.57" upper="1.57" effort="3.5" velocity="7.3" />
     </joint>
     <!-- Link C -->
@@ -114,5 +114,5 @@
       <child link="${leg_name}_linkC" />
       <axis xyz="0 0 1" />
-      <limit lower="-3.14" upper="1.57" effort="50" velocity="7.3" />
+      <limit lower="-3.14" upper="1.57" effort="3.5" velocity="7.3" />
     </joint>
     <!-- FCP Link -->

File: elkapod_description/urdf/right_leg/right_leg.urdf.xacro (robot description, xacro)
@@ -56,5 +56,5 @@
         <child link="${leg_name}_linkA" />
         <axis xyz="0 0 1" />
-        <limit lower="-1.57" upper="1.57" effort="50" velocity="7.3" />
+        <limit lower="-1.57" upper="1.57" effort="3.5" velocity="7.3" />
     </joint>
     <!-- Link B -->
@@ -85,5 +85,5 @@
         <child link="${leg_name}_linkB" />
         <axis xyz="0 0 1" />
-        <limit lower="-1.57" upper="1.57" effort="50" velocity="7.3" />
+        <limit lower="-1.57" upper="1.57" effort="3.5" velocity="7.3" />
     </joint>
     <!-- Link C -->
@@ -114,5 +114,5 @@
         <child link="${leg_name}_linkC" />
         <axis xyz="0 0 1" />
-        <limit lower="-3.14" upper="3.14" effort="50" velocity="7.3" />
+        <limit lower="-3.14" upper="3.14" effort="3.5" velocity="7.3" />
     </joint>
     <!-- FCP link -->

Commit message: #20 Moved locomotion system launch from bringup to motion manager launch, changed publish rate of ros2_controller

File: elkapod_description/urdf/left_leg/left_leg.urdf.xacro (robot description, xacro)
@@ -56,5 +56,5 @@
       <child link="${leg_name}_linkA" />
       <axis xyz="0 0 1" />
-      <limit lower="-1.57" upper="1.57" effort="3.5" velocity="7.3" />
+      <limit lower="-1.57" upper="1.57" effort="50.0" velocity="7.3" />
     </joint>
     <!-- Link B -->
@@ -85,5 +85,5 @@
       <child link="${leg_name}_linkB" />
       <axis xyz="0 0 1" />
-      <limit lower="-1.57" upper="1.57" effort="3.5" velocity="7.3" />
+      <limit lower="-1.57" upper="1.57" effort="50.0" velocity="7.3" />
     </joint>
     <!-- Link C -->
@@ -114,5 +114,5 @@
       <child link="${leg_name}_linkC" />
       <axis xyz="0 0 1" />
-      <limit lower="-3.14" upper="1.57" effort="3.5" velocity="7.3" />
+      <limit lower="-3.14" upper="1.57" effort="50.0" velocity="7.3" />
     </joint>
     <!-- FCP Link -->
@@ -140,6 +140,6 @@
     </link>
     <gazebo reference="${leg_name}_FCP">
-      <mu1>1000.0</mu1>
-      <mu2>1000.0</mu2>
+      <mu1>10.0</mu1>
+      <mu2>10.0</mu2>
     </gazebo>
     <!-- Fixed Joint for FCP -->

File: elkapod_description/urdf/right_leg/right_leg.urdf.xacro (robot description, xacro)
@@ -56,5 +56,5 @@
         <child link="${leg_name}_linkA" />
         <axis xyz="0 0 1" />
-        <limit lower="-1.57" upper="1.57" effort="3.5" velocity="7.3" />
+        <limit lower="-1.57" upper="1.57" effort="50.0" velocity="7.3" />
     </joint>
     <!-- Link B -->
@@ -85,5 +85,5 @@
         <child link="${leg_name}_linkB" />
         <axis xyz="0 0 1" />
-        <limit lower="-1.57" upper="1.57" effort="3.5" velocity="7.3" />
+        <limit lower="-1.57" upper="1.57" effort="50.0" velocity="7.3" />
     </joint>
     <!-- Link C -->
@@ -114,5 +114,5 @@
         <child link="${leg_name}_linkC" />
         <axis xyz="0 0 1" />
-        <limit lower="-3.14" upper="3.14" effort="3.5" velocity="7.3" />
+        <limit lower="-3.14" upper="3.14" effort="50.0" velocity="7.3" />
     </joint>
     <!-- FCP link -->
@@ -140,6 +140,6 @@
     </link>
     <gazebo reference="${leg_name}_FCP">
-      <mu1>1000.0</mu1>
-      <mu2>1000.0</mu2>
+      <mu1>10.0</mu1>
+      <mu2>10.0</mu2>
     </gazebo>
     <!-- Fixed joint for FCP -->

File: elkapod_description/urdf/ros2_control.xacro (robot description, xacro)
@@ -10,4 +10,6 @@
               <param name="initial_value">${initial_angle_rad}</param>
             </state_interface>
+            <state_interface name="velocity"/>
+            <state_interface name="effort"/>
         </joint>
     </xacro:macro>

Commit message: Walking stack v1.0.0 (#22)
* (#13)(#17) Implemented first gait controller prototype, added input to elkapod_leg_controller

* (#17) Fixed unstable base height during walking by adding smoothstep function for scaling in Z function of swing phase

* #17 Started work on adding angular velocity command

* #17 Corrected joint angle limits for the robot

* #17 Added launch file for whole system, further work on angular speed

* #17 Added friction coefficients to leg's toucher

* Added locomotion examples, added Odometry plugin for ground truth odom in GazeboSim

* #14 Added smooth transition from IDLE standing pose to walking with phase shift, other changes to gait generator

* #17 Replaced mesh foot with geometry sphere foot thus improving simulation speed and enabling friction

* #17 Added phase lag during start of swing phase

* #17 Added base height setting and fixed bug related to phase lag

* #17 Added on/off functionality for gait generator (behaviour similar to ros2_controller)

* #20 Started implementing elkapod_motion_manager along with light trajectory planner & executioner

* #20 Added init, standing up and lowering sequences to manager

* #17 Added elkapod_motion_manager to the launch file, changed effort in the joints to 3.5Nm, other minor changes

* #17 Translated gait generator into cpp (not working yet)

* #17 Fixed cpp gait generator, code refactoring and cleaning

* #20 Moved locomotion system launch from bringup to motion manager launch, changed publish rate of ros2_controller

* #20 Added action server to motion manager, services for walk transistions, other bug fixes

* Formatted all code using ruff and clang-format (google style)

* Updated CI

* Fixed angular velocity bug

* #13 Changed the name of the kinematics package, added NaN publishing prevention mechanism

* Fixed bug in the elkapod_motion_manager that caused all zeros being published during trajectory execution, other minor changes

* README.md update

File: elkapod_description/urdf/left_leg/left_leg.urdf.xacro (robot description, xacro)
@@ -56,5 +56,5 @@
       <child link="${leg_name}_linkA" />
       <axis xyz="0 0 1" />
-      <limit lower="-1.57" upper="1.57" effort="5" velocity="1.0" />
+      <limit lower="-1.57" upper="1.57" effort="50.0" velocity="7.3" />
     </joint>
     <!-- Link B -->
@@ -85,5 +85,5 @@
       <child link="${leg_name}_linkB" />
       <axis xyz="0 0 1" />
-      <limit lower="-1.57" upper="1.57" effort="5" velocity="1.0" />
+      <limit lower="-1.57" upper="1.57" effort="50.0" velocity="7.3" />
     </joint>
     <!-- Link C -->
@@ -114,5 +114,5 @@
       <child link="${leg_name}_linkC" />
       <axis xyz="0 0 1" />
-      <limit lower="-3.14" upper="1.57" effort="5" velocity="1.0" />
+      <limit lower="-3.14" upper="1.57" effort="50.0" velocity="7.3" />
     </joint>
     <!-- FCP Link -->
@@ -126,5 +126,5 @@
         <origin xyz="0 0 0" rpy="0 0 0" />
         <geometry>
-          <mesh filename="package://elkapod_description/meshes/left_leg/FCP.STL" />
+          <sphere radius="0.01"/>
         </geometry>
         <material name="">
@@ -135,8 +135,12 @@
         <origin xyz="0 0 0" rpy="0 0 0" />
         <geometry>
-          <mesh filename="package://elkapod_description/meshes/left_leg/FCP.STL" />
+          <sphere radius="0.01"/>
         </geometry>
       </collision>
     </link>
+    <gazebo reference="${leg_name}_FCP">
+      <mu1>10.0</mu1>
+      <mu2>10.0</mu2>
+    </gazebo>
     <!-- Fixed Joint for FCP -->
     <joint name="${leg_name}_FCP_joint" type="fixed">

File: elkapod_description/urdf/right_leg/right_leg.urdf.xacro (robot description, xacro)
@@ -56,5 +56,5 @@
         <child link="${leg_name}_linkA" />
         <axis xyz="0 0 1" />
-        <limit lower="-1.57" upper="1.57" effort="5" velocity="1.0" />
+        <limit lower="-1.57" upper="1.57" effort="50.0" velocity="7.3" />
     </joint>
     <!-- Link B -->
@@ -85,5 +85,5 @@
         <child link="${leg_name}_linkB" />
         <axis xyz="0 0 1" />
-        <limit lower="-1.57" upper="1.57" effort="5" velocity="1.0" />
+        <limit lower="-1.57" upper="1.57" effort="50.0" velocity="7.3" />
     </joint>
     <!-- Link C -->
@@ -114,5 +114,5 @@
         <child link="${leg_name}_linkC" />
         <axis xyz="0 0 1" />
-        <limit lower="-3.14" upper="3.14" effort="5" velocity="1.0" />
+        <limit lower="-3.14" upper="3.14" effort="50.0" velocity="7.3" />
     </joint>
     <!-- FCP link -->
@@ -126,5 +126,5 @@
         <origin xyz="0 0 0" rpy="0 0 0" />
         <geometry>
-          <mesh filename="package://elkapod_description/meshes/right_leg/FCP.STL" />
+          <sphere radius="0.01"/>
         </geometry>
         <material name="">
@@ -135,8 +135,12 @@
         <origin xyz="0 0 0" rpy="0 0 0" />
         <geometry>
-          <mesh filename="package://elkapod_description/meshes/right_leg/FCP.STL" />
+          <sphere radius="0.01"/>
         </geometry>
       </collision>
     </link>
+    <gazebo reference="${leg_name}_FCP">
+      <mu1>10.0</mu1>
+      <mu2>10.0</mu2>
+    </gazebo>
     <!-- Fixed joint for FCP -->
     <joint name="${leg_name}_FCP_joint" type="fixed">

File: elkapod_description/urdf/ros2_control.xacro (robot description, xacro)
@@ -10,4 +10,6 @@
               <param name="initial_value">${initial_angle_rad}</param>
             </state_interface>
+            <state_interface name="velocity"/>
+            <state_interface name="effort"/>
         </joint>
     </xacro:macro>
@@ -18,21 +20,21 @@
             </hardware>
             <xacro:joint_interface name="leg1_J1" min_pos_rad="-1.57" max_pos_rad="1.57" initial_angle_rad="0.0"/>
-            <xacro:joint_interface name="leg1_J2" min_pos_rad="-3.14" max_pos_rad="3.14" initial_angle_rad="0.0"/>
-            <xacro:joint_interface name="leg1_J3" min_pos_rad="-3.14" max_pos_rad="3.14" initial_angle_rad="0.0"/>
+            <xacro:joint_interface name="leg1_J2" min_pos_rad="-1.57" max_pos_rad="1.57" initial_angle_rad="0.0"/>
+            <xacro:joint_interface name="leg1_J3" min_pos_rad="-3.14" max_pos_rad="0.0" initial_angle_rad="0.0"/>
             <xacro:joint_interface name="leg3_J1" min_pos_rad="-1.57" max_pos_rad="1.57" initial_angle_rad="0.0"/>
-            <xacro:joint_interface name="leg3_J2" min_pos_rad="-3.14" max_pos_rad="3.14" initial_angle_rad="0.0"/>
-            <xacro:joint_interface name="leg3_J3" min_pos_rad="-3.14" max_pos_rad="3.14" initial_angle_rad="0.0"/>
+            <xacro:joint_interface name="leg3_J2" min_pos_rad="-1.57" max_pos_rad="1.57" initial_angle_rad="0.0"/>
+            <xacro:joint_interface name="leg3_J3" min_pos_rad="-3.14" max_pos_rad="0.0" initial_angle_rad="0.0"/>
             <xacro:joint_interface name="leg5_J1" min_pos_rad="-1.57" max_pos_rad="1.57" initial_angle_rad="0.0"/>
-            <xacro:joint_interface name="leg5_J2" min_pos_rad="-3.14" max_pos_rad="3.14" initial_angle_rad="0.0"/>
-            <xacro:joint_interface name="leg5_J3" min_pos_rad="-3.14" max_pos_rad="3.14" initial_angle_rad="0.0"/>
+            <xacro:joint_interface name="leg5_J2" min_pos_rad="-1.57" max_pos_rad="1.57" initial_angle_rad="0.0"/>
+            <xacro:joint_interface name="leg5_J3" min_pos_rad="-3.14" max_pos_rad="0.0" initial_angle_rad="0.0"/>
             <xacro:joint_interface name="leg2_J1" min_pos_rad="-1.57" max_pos_rad="1.57" initial_angle_rad="0.0"/>
-            <xacro:joint_interface name="leg2_J2" min_pos_rad="-3.14" max_pos_rad="3.14" initial_angle_rad="0.0"/>
-            <xacro:joint_interface name="leg2_J3" min_pos_rad="-3.14" max_pos_rad="3.14" initial_angle_rad="0.0"/>
+            <xacro:joint_interface name="leg2_J2" min_pos_rad="-1.57" max_pos_rad="1.57" initial_angle_rad="0.0"/>
+            <xacro:joint_interface name="leg2_J3" min_pos_rad="-3.14" max_pos_rad="0.0" initial_angle_rad="0.0"/>
             <xacro:joint_interface name="leg4_J1" min_pos_rad="-1.57" max_pos_rad="1.57" initial_angle_rad="0.0"/>
-            <xacro:joint_interface name="leg4_J2" min_pos_rad="-3.14" max_pos_rad="3.14" initial_angle_rad="0.0"/>
-            <xacro:joint_interface name="leg4_J3" min_pos_rad="-3.14" max_pos_rad="3.14" initial_angle_rad="0.0"/>
+            <xacro:joint_interface name="leg4_J2" min_pos_rad="-1.57" max_pos_rad="1.57" initial_angle_rad="0.0"/>
+            <xacro:joint_interface name="leg4_J3" min_pos_rad="-3.14" max_pos_rad="0.0" initial_angle_rad="0.0"/>
             <xacro:joint_interface name="leg6_J1" min_pos_rad="-1.57" max_pos_rad="1.57" initial_angle_rad="0.0"/>
-            <xacro:joint_interface name="leg6_J2" min_pos_rad="-3.14" max_pos_rad="3.14" initial_angle_rad="0.0"/>
-            <xacro:joint_interface name="leg6_J3" min_pos_rad="-3.14" max_pos_rad="3.14" initial_angle_rad="0.0"/>
+            <xacro:joint_interface name="leg6_J2" min_pos_rad="-1.57" max_pos_rad="1.57" initial_angle_rad="0.0"/>
+            <xacro:joint_interface name="leg6_J3" min_pos_rad="-3.14" max_pos_rad="0.0" initial_angle_rad="0.0"/>
         </ros2_control>
     </xacro:if>
@@ -42,4 +44,9 @@
             <parameters>$(find elkapod_description)/config/gaz_ros2_ctl_use_sim.yaml</parameters>
         </plugin>
+        <plugin filename="gz-sim-odometry-publisher-system" name="gz::sim::systems::OdometryPublisher">
+            <odom_frame>base_link</odom_frame>
+            <robot_base_frame>base_link</robot_base_frame>
+            <odom_publish_frequency>50</odom_publish_frequency>
+        </plugin>
     </gazebo>
 </robot>
