Commit message: #32 First version of force sensors added

File: elkapod_description/urdf/left_leg/left_leg.urdf.xacro (robot description, xacro)
@@ -143,10 +143,26 @@
       <mu2>10.0</mu2>
     </gazebo>
+    <gazebo reference="${leg_name}_FCP_joint">
+        <sensor name="${leg_name}_fsr" type="force_torque">
+          <always_on>true</always_on>
+          <update_rate>100</update_rate>
+          <visualize>true</visualize>
+          <topic>/legs/${leg_name}/fsr</topic>
+          <enable_metrics>true</enable_metrics>
+          <pose>0 0 0 0 0 0</pose>
+          <force_torque>
+            <frame>sensor</frame>
+            <measure_direction>child_to_parent</measure_direction>
+          </force_torque>
+        </sensor>
+    </gazebo>
     <!-- Fixed Joint for FCP -->
-    <joint name="${leg_name}_FCP_joint" type="fixed">
+    <joint name="${leg_name}_FCP_joint" type="prismatic">
       <origin xyz="0.2135 0.0085747 0" rpy="0 0 -0.29403" />
       <parent link="${leg_name}_linkC" />
       <child link="${leg_name}_FCP" />
-      <axis xyz="0 0 0" />
+      <axis xyz="1 0 0" />
+      <limit effort="1000.0" lower="-0.0001" upper="0.0001" velocity="30"/>
+      <dynamics damping="10.0" friction="0.0"/>
     </joint>
   </xacro:macro>

File: elkapod_description/urdf/right_leg/right_leg.urdf.xacro (robot description, xacro)
@@ -143,10 +143,26 @@
       <mu2>10.0</mu2>
     </gazebo>
+    <gazebo reference="${leg_name}_FCP_joint">
+        <sensor name="${leg_name}_fsr" type="force_torque">
+          <always_on>true</always_on>
+          <update_rate>100</update_rate>
+          <visualize>true</visualize>
+          <topic>/legs/${leg_name}/fsr</topic>
+          <enable_metrics>true</enable_metrics>
+          <pose>0 0 0 0 0 0</pose>
+          <force_torque>
+            <frame>sensor</frame>
+            <measure_direction>child_to_parent</measure_direction>
+          </force_torque>
+        </sensor>
+    </gazebo>
     <!-- Fixed joint for FCP -->
-    <joint name="${leg_name}_FCP_joint" type="fixed">
+    <joint name="${leg_name}_FCP_joint" type="prismatic">
         <origin xyz="0.213503787197785 0.00857470533092818 0" rpy="0 0 -0.294032099334707" />
         <parent link="${leg_name}_linkC" />
         <child link="${leg_name}_FCP" />
-        <axis xyz="0 0 0" />
+        <axis xyz="1 0 0" />
+        <limit effort="1000.0" lower="-0.0001" upper="0.0001" velocity="30"/>
+        <dynamics damping="10.0" friction="0.0"/>
     </joint>
   </xacro:macro>

Commit message: Replaced force sensors in simulation with contact sensors, added PID controllers for pitch and roll control (to be tuned)

File: elkapod_description/urdf/left_leg/left_leg.urdf.xacro (robot description, xacro)
@@ -132,5 +132,5 @@
         </material>
       </visual>
-      <collision>
+      <collision name="${leg_name}_FCP">
         <origin xyz="0 0 0" rpy="0 0 0" />
         <geometry>
@@ -146,5 +146,5 @@
       <minDepth>0.01</minDepth>
     </gazebo>
-    <gazebo reference="${leg_name}_FCP_joint">
+    <!-- <gazebo reference="${leg_name}_FCP_joint">
         <sensor name="${leg_name}_fsr" type="force_torque">
           <always_on>true</always_on>
@@ -159,4 +159,14 @@
           </force_torque>
         </sensor>
+    </gazebo> -->
+    <gazebo reference="${leg_name}_FCP">
+      <sensor name="contact" type="contact">
+        <always_on>true</always_on>
+        <update_rate>100</update_rate>
+        <contact>
+          <collision>${leg_name}_FCP_collision</collision>
+        </contact>
+        <topic>/legs/${leg_name}_fsr</topic>
+      </sensor>
     </gazebo>
     <!-- Fixed Joint for FCP -->

File: elkapod_description/urdf/right_leg/right_leg.urdf.xacro (robot description, xacro)
@@ -132,5 +132,5 @@
         </material>
       </visual>
-      <collision>
+      <collision name="${leg_name}_FCP">
         <origin xyz="0 0 0" rpy="0 0 0" />
         <geometry>
@@ -146,5 +146,5 @@
       <minDepth>0.01</minDepth>
     </gazebo>
-    <gazebo reference="${leg_name}_FCP_joint">
+    <!-- <gazebo reference="${leg_name}_FCP_joint">
         <sensor name="${leg_name}_fsr" type="force_torque">
           <always_on>true</always_on>
@@ -159,4 +159,14 @@
           </force_torque>
         </sensor>
+    </gazebo> -->
+    <gazebo reference="${leg_name}_FCP">
+      <sensor name="contact" type="contact">
+        <always_on>true</always_on>
+        <update_rate>100</update_rate>
+        <contact>
+          <collision>${leg_name}_FCP_collision</collision>
+        </contact>
+        <topic>/legs/${leg_name}_fsr</topic>
+      </sensor>
     </gazebo>
     <!-- Fixed joint for FCP -->
