Commit message: #28 Merged ros2_control.xacro files into single one with sim_mode param

File: elkapod_description/urdf/elkapod.urdf.xacro (robot description, xacro)
@@ -2,7 +2,5 @@
 <robot xmlns:xacro="http://ros.org/wiki/xacro" name="elkapod">
   <!-- Execution env config -->
-  <xacro:arg name="use_sim_time" default="false"/>
-  <!-- Execution env configuration -->
-  <xacro:property name="use_sim_time" default="$(arg use_sim_time)"/>
+  <xacro:arg name="sim_mode" default="false"/>
   <!-- INCLUDES -->
   <!-- Colors -->
@@ -19,6 +17,6 @@
   <xacro:leg_right leg_name="leg4" parent="base_link" pos_x="0.0138" pos_y="-0.1643" pos_z="-0.03" roll="0" pitch="0" yaw="-1.57"/>
   <xacro:leg_right leg_name="leg6" parent="base_link" pos_x="-0.15903" pos_y="-0.15038" pos_z="-0.03" roll="0" pitch="0" yaw="-2.384143643587"/>
-  <xacro:include filename="$(find elkapod_description)/urdf/imu.xacro" />
   <!-- ros2_control -->
-  <xacro:include filename="$(find elkapod_description)/ros2_control/legs_system.ros2_control.xacro" />
+  <xacro:include filename="$(find elkapod_description)/ros2_control/elkapod.ros2_control.xacro" />
+  <xacro:elkapod_ros2_control sim_mode="$(arg sim_mode)"/>
 </robot>

Commit message: Hardware interfaces v1.0.0 (#26)
* #23 Started working on hardware interface implemenation

* #23 First version of somehow working hardware interface

* #23 Tested cleaner write method

* #23 Started implementing SPI communication

* #23 Parameters parsing inside on_init, added temperature sensor interface, added start and shutdown messages via UART

* #23 Added temperature and battery info publishing, fixed some bugs, added declared command and state interfaces validation

* #23 Added IMU sensor to hardware interface and IMU Broadcaster

* #23 Added connection checking via UART and port closing after crash in on_error() method

* #23 Formatted code

* Updated CI workflow

* #28 Merged ros2_control.xacro files into single one with sim_mode param

* Closes #28, cleaned launch files

* fixes #27

File: elkapod_description/urdf/elkapod.urdf.xacro (robot description, xacro)
@@ -2,7 +2,5 @@
 <robot xmlns:xacro="http://ros.org/wiki/xacro" name="elkapod">
   <!-- Execution env config -->
-  <xacro:arg name="use_sim_time" default="false"/>
-  <!-- Execution env configuration -->
-  <xacro:property name="use_sim_time" default="$(arg use_sim_time)"/>
+  <xacro:arg name="sim_mode" default="false"/>
   <!-- INCLUDES -->
   <!-- Colors -->
@@ -19,6 +17,6 @@
   <xacro:leg_right leg_name="leg4" parent="base_link" pos_x="0.0138" pos_y="-0.1643" pos_z="-0.03" roll="0" pitch="0" yaw="-1.57"/>
   <xacro:leg_right leg_name="leg6" parent="base_link" pos_x="-0.15903" pos_y="-0.15038" pos_z="-0.03" roll="0" pitch="0" yaw="-2.384143643587"/>
-  <xacro:include filename="$(find elkapod_description)/urdf/imu.xacro" />
   <!-- ros2_control -->
-  <xacro:include filename="$(find elkapod_description)/urdf/ros2_control.xacro" />
+  <xacro:include filename="$(find elkapod_description)/ros2_control/elkapod.ros2_control.xacro" />
+  <xacro:elkapod_ros2_control sim_mode="$(arg sim_mode)"/>
 </robot>

Commit message: Removed imu xacro file Added sim macros for sensors

File: elkapod_description/urdf/elkapod.urdf.xacro (robot description, xacro)
@@ -20,4 +20,6 @@
   <xacro:include filename="$(find elkapod_description)/urdf/sensors/lidar.xacro" />
   <xacro:include filename="$(find elkapod_description)/urdf/sensors/depth_camera.xacro" />
+  <xacro:elkapod_sensors_lidar sim_mode="$(arg sim_mode)"/>
+  <xacro:elkapod_sensors_fron_camera sim_mode="$(arg sim_mode)"/>
   <!-- ros2_control -->
   <xacro:include filename="$(find elkapod_description)/ros2_control/elkapod.ros2_control.xacro" />

File: elkapod_description/urdf/sensors/depth_camera.xacro (robot description, xacro)
@@ -35,32 +35,36 @@
         <axis xyz="0 0 0" />
     </joint>
-    <gazebo reference="front_camera_optical">
-        <sensor name="camera" type="rgbd_camera">
-            <pose> 0 0 0 0 0 0 </pose>
-            <topic>front_camera</topic>
-            <visualize>true</visualize>
-            <update_rate>30</update_rate>
-            <always_on>true</always_on>
-            <camera>
-                <horizontal_fov>1.20428</horizontal_fov>
-                <image>
-                    <format>R8G8B8</format>
-                    <width>640</width>
-                    <height>480</height>
-                </image>
-                <clip>
-                    <near>0.1</near>
-                    <far>30</far>
-                </clip>
-                <depth_camera>
-                    <output>depths</output>
-                    <clip>
-                        <near>0.1</near>
-                        <far>30</far>
-                    </clip>
-                </depth_camera>
-            </camera>
-            <gz_frame_id>front_camera_optical</gz_frame_id>
-        </sensor>
-    </gazebo>
+    <xacro:macro name="elkapod_sensors_fron_camera" params="sim_mode:=^|false">
+        <xacro:if value="${sim_mode}">
+            <gazebo reference="front_camera_optical">
+                <sensor name="camera" type="rgbd_camera">
+                    <pose> 0 0 0 0 0 0 </pose>
+                    <topic>front_camera</topic>
+                    <visualize>true</visualize>
+                    <update_rate>30</update_rate>
+                    <always_on>true</always_on>
+                    <camera>
+                        <horizontal_fov>1.20428</horizontal_fov>
+                        <image>
+                            <format>R8G8B8</format>
+                            <width>640</width>
+                            <height>480</height>
+                        </image>
+                        <clip>
+                            <near>0.1</near>
+                            <far>30</far>
+                        </clip>
+                        <depth_camera>
+                            <output>depths</output>
+                            <clip>
+                                <near>0.1</near>
+                                <far>30</far>
+                            </clip>
+                        </depth_camera>
+                    </camera>
+                    <gz_frame_id>front_camera_optical</gz_frame_id>
+                </sensor>
+            </gazebo>
+        </xacro:if>
+    </xacro:macro>
 </robot>

File: elkapod_description/urdf/sensors/lidar.xacro (robot description, xacro)
@@ -35,39 +35,43 @@
         <axis xyz="0 0 0" />
     </joint>
-    <gazebo reference="lidar_optical">
-        <sensor name="lidar" type="gpu_lidar">
-            <always_on>true</always_on>
-            <!-- Downgraded values, so your GPU doesn't melt -->
-            <!-- <update_rate>10</update_rate> -->
-            <update_rate>3</update_rate>
-            <visualize>true</visualize>
-            <topic>lidar_data</topic>
-            <lidar>
-                <scan>
-                    <horizontal>
-                        <!-- Downgraded values, so your GPU doesn't melt -->
-                        <!-- <samples>900</samples> -->
-                        <samples>90</samples>
-                        <resolution>1</resolution>
-                        <min_angle>-3.14</min_angle>
-                        <max_angle>3.14</max_angle>
-                    </horizontal>
-                    <vertical>
-                        <!-- Downgraded values, so your GPU doesn't melt -->
-                        <samples>25</samples>
-                        <!-- <samples>95</samples> -->
-                        <resolution>1</resolution>
-                        <min_angle>0</min_angle>
-                        <max_angle>1.57079633</max_angle>
-                    </vertical>
-                </scan>
-                <range>
-                    <min>0.1</min>
-                    <max>30</max>
-                    <resolution>0.01</resolution>
-                </range>
-            </lidar>
-            <gz_frame_id>lidar_optical</gz_frame_id>
-        </sensor>
-    </gazebo>
+    <xacro:macro name="elkapod_sensors_lidar" params="sim_mode:=^|false">
+        <xacro:if value="${sim_mode}">
+            <gazebo reference="lidar_optical">
+                <sensor name="lidar" type="gpu_lidar">
+                    <always_on>true</always_on>
+                    <!-- Downgraded values, so your GPU doesn't melt -->
+                    <!-- <update_rate>10</update_rate> -->
+                    <update_rate>3</update_rate>
+                    <visualize>true</visualize>
+                    <topic>lidar_data</topic>
+                    <lidar>
+                        <scan>
+                            <horizontal>
+                                <!-- Downgraded values, so your GPU doesn't melt -->
+                                <!-- <samples>900</samples> -->
+                                <samples>90</samples>
+                                <resolution>1</resolution>
+                                <min_angle>-3.14</min_angle>
+                                <max_angle>3.14</max_angle>
+                            </horizontal>
+                            <vertical>
+                                <!-- Downgraded values, so your GPU doesn't melt -->
+                                <samples>25</samples>
+                                <!-- <samples>95</samples> -->
+                                <resolution>1</resolution>
+                                <min_angle>0</min_angle>
+                                <max_angle>1.57079633</max_angle>
+                            </vertical>
+                        </scan>
+                        <range>
+                            <min>0.1</min>
+                            <max>30</max>
+                            <resolution>0.01</resolution>
+                        </range>
+                    </lidar>
+                    <gz_frame_id>lidar_optical</gz_frame_id>
+                </sensor>
+            </gazebo>
+        </xacro:if>
+    </xacro:macro>
 </robot>

Commit message: added some xacros adjusting lidar work in simulation

File: elkapod_description/urdf/elkapod.urdf.xacro (robot description, xacro)
@@ -18,7 +18,12 @@
   <xacro:leg_right leg_name="leg6" parent="base_link" pos_x="-0.15903" pos_y="-0.15038" pos_z="-0.03" roll="0" pitch="0" yaw="-2.384143643587"/>
   <!-- Sensors -->
+  <xacro:arg name="lidar_mode" default="minimal"/>
+   <xacro:arg name="lidar_rate" default="10"/>
   <xacro:include filename="$(find elkapod_description)/urdf/sensors/lidar.xacro" />
   <xacro:include filename="$(find elkapod_description)/urdf/sensors/depth_camera.xacro" />
-  <xacro:elkapod_sensors_lidar sim_mode="$(arg sim_mode)"/>
+  <xacro:elkapod_sensors_lidar
+      sim_mode="$(arg sim_mode)"
+      lidar_mode="$(arg lidar_mode)"
+      lidar_rate="$(arg lidar_rate)"/>
   <xacro:elkapod_sensors_fron_camera sim_mode="$(arg sim_mode)"/>
   <!-- ros2_control -->

File: elkapod_description/urdf/sensors/lidar.xacro (robot description, xacro)
@@ -35,42 +35,41 @@
         <axis xyz="0 0 0" />
     </joint>
-    <xacro:macro name="elkapod_sensors_lidar" params="sim_mode:=^|false">
+    <xacro:macro name="elkapod_sensors_lidar"
+     params="sim_mode:=^|false lidar_mode:=minimal lidar_rate:=5">
         <xacro:if value="${sim_mode}">
-            <gazebo reference="lidar_optical">
-                <sensor name="lidar" type="gpu_lidar">
-                    <always_on>true</always_on>
-                    <!-- Downgraded values, so your GPU doesn't melt -->
-                    <!-- <update_rate>10</update_rate> -->
-                    <update_rate>3</update_rate>
-                    <visualize>true</visualize>
-                    <topic>lidar_data</topic>
-                    <lidar>
-                        <scan>
-                            <horizontal>
-                                <!-- Downgraded values, so your GPU doesn't melt -->
-                                <!-- <samples>900</samples> -->
-                                <samples>90</samples>
-                                <resolution>1</resolution>
-                                <min_angle>-3.14</min_angle>
-                                <max_angle>3.14</max_angle>
-                            </horizontal>
-                            <vertical>
-                                <!-- Downgraded values, so your GPU doesn't melt -->
-                                <samples>25</samples>
-                                <!-- <samples>95</samples> -->
-                                <resolution>1</resolution>
-                                <min_angle>0</min_angle>
-                                <max_angle>1.57079633</max_angle>
-                            </vertical>
-                        </scan>
-                        <range>
-                            <min>0.1</min>
-                            <max>30</max>
-                            <resolution>0.01</resolution>
-                        </range>
-                    </lidar>
-                    <gz_frame_id>lidar_optical</gz_frame_id>
-                </sensor>
-            </gazebo>
+            <xacro:unless value="${lidar_mode == 'off'}">
+                <xacro:property name="h_samples" value="${600 if lidar_mode == 'full' else 120}"/>
+                <xacro:property name="v_samples" value="${95 if lidar_mode == 'full' else 25}"/>
+                <gazebo reference="lidar_optical">
+                    <sensor name="lidar" type="gpu_lidar">
+                        <always_on>true</always_on>
+                        <update_rate>${lidar_rate}</update_rate>
+                        <visualize>true</visualize>
+                        <topic>lidar_data</topic>
+                        <lidar>
+                            <scan>
+                                <horizontal>
+                                    <samples>${h_samples}</samples>
+                                    <resolution>1</resolution>
+                                    <min_angle>-3.14</min_angle>
+                                    <max_angle>3.14</max_angle>
+                                </horizontal>
+                                <vertical>
+                                    <samples>${v_samples}</samples>
+                                    <resolution>1</resolution>
+                                    <min_angle>0</min_angle>
+                                    <max_angle>1.57079633</max_angle>
+                                </vertical>
+                            </scan>
+                            <range>
+                                <min>0.1</min>
+                                <max>30</max>
+                                <resolution>0.01</resolution>
+                            </range>
+                        </lidar>
+                        <gz_frame_id>lidar_optical</gz_frame_id>
+                    </sensor>
+                </gazebo>
+            </xacro:unless>
         </xacro:if>
     </xacro:macro>
